File: Backplane/Backplane.sch (KiCad schematic (older format))
At the start: 3 parts

Commit message: Long overdue update...
Parts:
- removed J?: Conn_02x35_Odd_Even, symbol Connector_Generic:Conn_02x35_Odd_Even
- removed J?: Conn_02x25_Odd_Even, symbol Connector_Generic:Conn_02x25_Odd_Even
- added C1, C3: 220uF 100V, Capacitor_THT:CP_Radial_D7.5mm_P2.50mm, symbol Device:CP
- added C2: 470uF 6.3V, Capacitor_THT:CP_Radial_D7.5mm_P2.50mm, symbol Device:CP
- added C4: 0.1uF, Capacitor_THT:C_Disc_D3.0mm_W2.0mm_P2.50mm, symbol Device:C
- added D1, D2: SA5.0CA-E3/54, Diode_THT:D_DO-15_P12.70mm_Horizontal, symbol Device:D_TVS_ALT
- added D10, D11, D12, D13, D14, D15, D16, D17, D18, D19, D20, D21, D22, D23, D24, D25, D26, D27, D28, D29, D30, D31, D32, D33, D34, D35, D36, D37, D38, D39, D4, D40, D41, D42, D43, D44, D45, D46, D47, D48, D49, D5, D50, D51, D6, D7, D8, D9: PESD5V0V1BA, Diode_SMD:D_SOD-323_HandSoldering, symbol Device:D_TVS_ALT
- added D3: POWER, LED_THT:LED_D3.0mm, symbol Device:LED
- added D53: SA12CA, Diode_THT:D_DO-15_P12.70mm_Horizontal, symbol Device:D_TVS_ALT
- added F1: MF-R600-2, Fuse:Fuse_Bourns_MF-RG600, symbol Device:Fuse
- added H1, H2, H3, H4, H5, H6: MountingHole_Pad, MountingHole:MountingHole_3.2mm_M3, symbol Mechanical:MountingHole_Pad
- added J10, J11, J9: Conn_02x25_Top_Bottom, CPCModular:Edge_Socket_2x25_2.54PS, symbol Connector_Generic:Conn_02x25_Top_Bottom
- added J12: Expansion Top (Edge connector), CPCModular:Edge25_2.54PS, symbol Connector:Conn_01x25_Male
- added J13: Expansion Bottom (Edge connector), CPCModular:Edge25_2.54PS, symbol Connector:Conn_01x25_Male
- added J14: USB_B, Connector_USB:USB_B_OST_USB-B1HSxx_Horizontal, symbol Connector:USB_B
- added J15: TE 171826-4 ('Berg'), Connector_JST:JST_EH_S4B-EH_1x04_P2.50mm_Horizontal, symbol Connector:Conn_01x04_Female
- added J16: Barrel_Jack_MountingPin, Connector_BarrelJack:BarrelJack_Horizontal, symbol Connector:Barrel_Jack_MountingPin
- added J17: SCART POWER, Connector_PinHeader_2.54mm:PinHeader_1x02_P2.54mm_Horizontal, symbol Connector:Conn_01x02_Male
- added J18: TE 770997-1 ('Molex'), Connector_JST:JST_EH_S4B-EH_1x04_P2.50mm_Horizontal, symbol Connector:Conn_01x04_Female
- added J2, J3, J4: Conn_02x25_Odd_Even, Connector_PinSocket_2.54mm:PinSocket_2x25_P2.54mm_Vertical, symbol Connector_Generic:Conn_02x25_Odd_Even
- added J5, J6, J7, J8: Conn_02x36_Top_Bottom, CPCModular:Edge_Socket_2x36_2.54PS, symbol Connector_Generic:Conn_02x36_Top_Bottom
- added R1: 470, Resistor_THT:R_Axial_DIN0207_L6.3mm_D2.5mm_P7.62mm_Horizontal, symbol Device:R
- added SW1: SSP1S1M6xEA, CPCModular:E-Switch_SSP1_M6_A, symbol Switch:SW_SPDT
- added SW2: PTS645VH58-2 LFS, Button_Switch_THT:SW_Tactile_SPST_Angled_PTS645Vx58-2LFS, symbol Switch:SW_Push
- added TH1: B57238S0709M000, Varistor:RV_Disc_D15.5mm_W5.9mm_P7.5mm, symbol Device:Thermistor_NTC
- added U1: RS6-0505S, CPCModular:Recom_RS6_Series_SIP8, symbol CPCModular:RS6-0505S
- added U2: ADM708 or MAX708, Package_DIP:DIP-8_W7.62mm_Socket, symbol CPCModular:ADM708
- added U3: TMU 3-0512, Converter_DCDC:Converter_DCDC_muRata_CRE1xxxxxxSC_THT, symbol Regulator_Switching:CRE1S2412SC
- J1: renamed from J?; footprint (none) -> Connector_PinSocket_2.54mm:PinSocket_2x25_P2.54mm_Vertical
Connections:
- net A0: now also J1.18 (Pin_18), D35.1 (A1), J13.9 (Pin_9), J2.18 (Pin_18), J3.18 (Pin_18), J4.18 (Pin_18), J5.46 (Pin_46), J6.46 (Pin_46), J7.46 (Pin_46), J8.46 (Pin_46)
- net A1: now also J1.17 (Pin_17), D12.1 (A1), J12.9 (Pin_9), J2.17 (Pin_17), J3.17 (Pin_17), J4.17 (Pin_17), J5.10 (Pin_10), J6.10 (Pin_10), J7.10 (Pin_10), J8.10 (Pin_10)
- net A10: now also J1.8 (Pin_8), D30.1 (A1), J10.32 (Pin_32), J11.32 (Pin_32), J13.4 (Pin_4), J2.8 (Pin_8), J3.8 (Pin_8), J4.8 (Pin_8), J5.41 (Pin_41), J6.41 (Pin_41), J7.41 (Pin_41), J8.41 (Pin_41), J9.32 (Pin_32)
- net A11: now also J1.7 (Pin_7), D7.1 (A1), J10.7 (Pin_7), J11.7 (Pin_7), J12.4 (Pin_4), J2.7 (Pin_7), J3.7 (Pin_7), J4.7 (Pin_7), J5.5 (Pin_5), J6.5 (Pin_5), J7.5 (Pin_5), J8.5 (Pin_5), J9.7 (Pin_7)
- net A12: now also J1.6 (Pin_6), D29.1 (A1), J10.31 (Pin_31), J11.31 (Pin_31), J13.3 (Pin_3), J2.6 (Pin_6), J3.6 (Pin_6), J4.6 (Pin_6), J5.40 (Pin_40), J6.40 (Pin_40), J7.40 (Pin_40), J8.40 (Pin_40), J9.31 (Pin_31)
- net A13: now also J1.5 (Pin_5), D6.1 (A1), J10.6 (Pin_6), J11.6 (Pin_6), J12.3 (Pin_3), J2.5 (Pin_5), J3.5 (Pin_5), J4.5 (Pin_5), J5.4 (Pin_4), J6.4 (Pin_4), J7.4 (Pin_4), J8.4 (Pin_4), J9.6 (Pin_6)
- net A14: now also J1.4 (Pin_4), D28.1 (A1), J10.30 (Pin_30), J11.30 (Pin_30), J13.2 (Pin_2), J2.4 (Pin_4), J3.4 (Pin_4), J4.4 (Pin_4), J5.39 (Pin_39), J6.39 (Pin_39), J7.39 (Pin_39), J8.39 (Pin_39), J9.30 (Pin_30)
- net A15: now also J1.3 (Pin_3), D5.1 (A1), J10.5 (Pin_5), J11.5 (Pin_5), J12.2 (Pin_2), J2.3 (Pin_3), J3.3 (Pin_3), J4.3 (Pin_3), J5.3 (Pin_3), J6.3 (Pin_3), J7.3 (Pin_3), J8.3 (Pin_3), J9.5 (Pin_5)
- net A2: now also J1.16 (Pin_16), D34.1 (A1), J13.8 (Pin_8), J2.16 (Pin_16), J3.16 (Pin_16), J4.16 (Pin_16), J5.45 (Pin_45), J6.45 (Pin_45), J7.45 (Pin_45), J8.45 (Pin_45)
- net A3: now also J1.15 (Pin_15), D11.1 (A1), J12.8 (Pin_8), J2.15 (Pin_15), J3.15 (Pin_15), J4.15 (Pin_15), J5.9 (Pin_9), J6.9 (Pin_9), J7.9 (Pin_9), J8.9 (Pin_9)
- net A4: now also J1.14 (Pin_14), D33.1 (A1), J13.7 (Pin_7), J2.14 (Pin_14), J3.14 (Pin_14), J4.14 (Pin_14), J5.44 (Pin_44), J6.44 (Pin_44), J7.44 (Pin_44), J8.44 (Pin_44)
- net A5: now also J1.13 (Pin_13), D10.1 (A1), J12.7 (Pin_7), J2.13 (Pin_13), J3.13 (Pin_13), J4.13 (Pin_13), J5.8 (Pin_8), J6.8 (Pin_8), J7.8 (Pin_8), J8.8 (Pin_8)
- net A6: now also J1.12 (Pin_12), D32.1 (A1), J13.6 (Pin_6), J2.12 (Pin_12), J3.12 (Pin_12), J4.12 (Pin_12), J5.43 (Pin_43), J6.43 (Pin_43), J7.43 (Pin_43), J8.43 (Pin_43)
- net A7: now also J1.11 (Pin_11), D9.1 (A1), J12.6 (Pin_6), J2.11 (Pin_11), J3.11 (Pin_11), J4.11 (Pin_11), J5.7 (Pin_7), J6.7 (Pin_7), J7.7 (Pin_7), J8.7 (Pin_7)
- net A8: now also J1.10 (Pin_10), D31.1 (A1), J10.33 (Pin_33), J11.33 (Pin_33), J13.5 (Pin_5), J2.10 (Pin_10), J3.10 (Pin_10), J4.10 (Pin_10), J5.42 (Pin_42), J6.42 (Pin_42), J7.42 (Pin_42), J8.42 (Pin_42), J9.33 (Pin_33)
- net A9: now also J1.9 (Pin_9), D8.1 (A1), J10.8 (Pin_8), J11.8 (Pin_8), J12.5 (Pin_5), J2.9 (Pin_9), J3.9 (Pin_9), J4.9 (Pin_9), J5.6 (Pin_6), J6.6 (Pin_6), J7.6 (Pin_6), J8.6 (Pin_6), J9.8 (Pin_8)
- net BC1: now also J10.44 (Pin_44), J11.44 (Pin_44), J9.44 (Pin_44)
- net BDIR: now also J10.43 (Pin_43), J11.43 (Pin_43), J9.43 (Pin_43)
- net CASRD: now also J10.2 (Pin_2), J11.2 (Pin_2), J9.2 (Pin_2)
- net CASWR: now also J10.27 (Pin_27), J11.27 (Pin_27), J9.27 (Pin_27)
- net CLK4: now also J1.50 (Pin_50), D51.1 (A1), J13.25 (Pin_25), J2.50 (Pin_50), J3.50 (Pin_50), J4.50 (Pin_50), J5.56 (Pin_56), J6.56 (Pin_56), J7.56 (Pin_56), J8.56 (Pin_56)
- net CURSOR: now also J1.46 (Pin_46), D49.1 (A1), J13.23 (Pin_23), J2.46 (Pin_46), J3.46 (Pin_46), J4.46 (Pin_46), J5.55 (Pin_55), J6.55 (Pin_55), J7.55 (Pin_55), J8.55 (Pin_55)
- net D0: now also J1.26 (Pin_26), D39.1 (A1), J10.41 (Pin_41), J11.41 (Pin_41), J13.13 (Pin_13), J2.26 (Pin_26), J3.26 (Pin_26), J4.26 (Pin_26), J5.50 (Pin_50), J6.50 (Pin_50), J7.50 (Pin_50), J8.50 (Pin_50), J9.41 (Pin_41)
- net D1: now also J1.25 (Pin_25), D16.1 (A1), J10.16 (Pin_16), J11.16 (Pin_16), J12.13 (Pin_13), J2.25 (Pin_25), J3.25 (Pin_25), J4.25 (Pin_25), J5.14 (Pin_14), J6.14 (Pin_14), J7.14 (Pin_14), J8.14 (Pin_14), J9.16 (Pin_16)
- net D2: now also J1.24 (Pin_24), D38.1 (A1), J10.40 (Pin_40), J11.40 (Pin_40), J13.12 (Pin_12), J2.24 (Pin_24), J3.24 (Pin_24), J4.24 (Pin_24), J5.49 (Pin_49), J6.49 (Pin_49), J7.49 (Pin_49), J8.49 (Pin_49), J9.40 (Pin_40)
- net D3: now also J1.23 (Pin_23), D15.1 (A1), J10.15 (Pin_15), J11.15 (Pin_15), J12.12 (Pin_12), J2.23 (Pin_23), J3.23 (Pin_23), J4.23 (Pin_23), J5.13 (Pin_13), J6.13 (Pin_13), J7.13 (Pin_13), J8.13 (Pin_13), J9.15 (Pin_15)
- net D4: now also J1.22 (Pin_22), D37.1 (A1), J10.39 (Pin_39), J11.39 (Pin_39), J13.11 (Pin_11), J2.22 (Pin_22), J3.22 (Pin_22), J4.22 (Pin_22), J5.48 (Pin_48), J6.48 (Pin_48), J7.48 (Pin_48), J8.48 (Pin_48), J9.39 (Pin_39)
- net D5: now also J1.21 (Pin_21), D14.1 (A1), J10.14 (Pin_14), J11.14 (Pin_14), J12.11 (Pin_11), J2.21 (Pin_21), J3.21 (Pin_21), J4.21 (Pin_21), J5.12 (Pin_12), J6.12 (Pin_12), J7.12 (Pin_12), J8.12 (Pin_12), J9.14 (Pin_14)
- net D6: now also J1.20 (Pin_20), D36.1 (A1), J10.38 (Pin_38), J11.38 (Pin_38), J13.10 (Pin_10), J2.20 (Pin_20), J3.20 (Pin_20), J4.20 (Pin_20), J5.47 (Pin_47), J6.47 (Pin_47), J7.47 (Pin_47), J8.47 (Pin_47), J9.38 (Pin_38)
- net D7: now also J1.19 (Pin_19), D13.1 (A1), J10.13 (Pin_13), J11.13 (Pin_13), J12.10 (Pin_10), J2.19 (Pin_19), J3.19 (Pin_19), J4.19 (Pin_19), J5.11 (Pin_11), J6.11 (Pin_11), J7.11 (Pin_11), J8.11 (Pin_11), J9.13 (Pin_13)
- net DISPEN: now also J5.27 (Pin_27), J6.27 (Pin_27), J7.27 (Pin_27), J8.27 (Pin_27)
- net GND: now also J1.2 (Pin_2), J1.49 (Pin_49), C2.2, C3.2, C4.2, D10.2 (A2), D11.2 (A2), D12.2 (A2), D13.2 (A2), D14.2 (A2), D15.2 (A2), D16.2 (A2), D17.2 (A2), D18.2 (A2), D19.2 (A2), D2.2 (A2), D20.2 (A2), D21.2 (A2), D22.2 (A2), D23.2 (A2), D24.2 (A2), D25.2 (A2), D26.2 (A2), D27.2 (A2), D28.2 (A2), D29.2 (A2), D3.1 (K), D30.2 (A2), D31.2 (A2), D32.2 (A2), D33.2 (A2), D34.2 (A2), D35.2 (A2), D36.2 (A2), D37.2 (A2), D38.2 (A2), D39.2 (A2), D4.2 (A2), D40.2 (A2), D41.2 (A2), D42.2 (A2), D43.2 (A2), D44.2 (A2), D45.2 (A2), D46.2 (A2), D47.2 (A2), D48.2 (A2), D49.2 (A2), D5.2 (A2), D50.2 (A2), D51.2 (A2), D53.2 (A2), D6.2 (A2), D7.2 (A2), D8.2 (A2), D9.2 (A2), H1.1, H2.1, H3.1, H4.1, H5.1, H6.1, J10.25 (Pin_25), J10.26 (Pin_26), J10.29 (Pin_29), J10.4 (Pin_4), J11.25 (Pin_25), J11.26 (Pin_26), J11.29 (Pin_29), J11.4 (Pin_4), J12.25 (Pin_25), J13.1 (Pin_1), J15.2 (Pin_2), J15.3 (Pin_3), J17.1 (Pin_1), J2.2 (Pin_2), J2.49 (Pin_49), J3.2 (Pin_2), J3.49 (Pin_49), J4.2 (Pin_2), J4.49 (Pin_49), J5.36 (Pin_36), J5.37 (Pin_37), J6.36 (Pin_36), J6.37 (Pin_37), J7.36 (Pin_36), J7.37 (Pin_37), J8.36 (Pin_36), J8.37 (Pin_37), J9.25 (Pin_25), J9.26 (Pin_26), J9.29 (Pin_29), J9.4 (Pin_4), SW2.2, U1.7 (Vout-), U2.3 (GND), U3.1 (-VIN), U3.3 (-VOUT)
- net HSYNC: now also J5.26 (Pin_26), J6.26 (Pin_26), J7.26 (Pin_26), J8.26 (Pin_26)
- net LEFT: now also J10.3 (Pin_3), J11.3 (Pin_3), J9.3 (Pin_3)
- net LPEN: now also J1.47 (Pin_47), D27.1 (A1), J12.24 (Pin_24), J2.47 (Pin_47), J3.47 (Pin_47), J4.47 (Pin_47), J5.24 (Pin_24), J6.24 (Pin_24), J7.24 (Pin_24), J8.24 (Pin_24)
- net MOTOR: now also J10.45 (Pin_45), J11.45 (Pin_45), J9.45 (Pin_45)
- net PA0: now also J10.34 (Pin_34), J11.34 (Pin_34), J9.34 (Pin_34)
- net PA1: now also J10.9 (Pin_9), J11.9 (Pin_9), J9.9 (Pin_9)
- net PA2: now also J10.35 (Pin_35), J11.35 (Pin_35), J9.35 (Pin_35)
- net PA3: now also J10.10 (Pin_10), J11.10 (Pin_10), J9.10 (Pin_10)
- net PA4: now also J10.36 (Pin_36), J11.36 (Pin_36), J9.36 (Pin_36)
- net PA5: now also J10.11 (Pin_11), J11.11 (Pin_11), J9.11 (Pin_11)
- net PA6: now also J10.37 (Pin_37), J11.37 (Pin_37), J9.37 (Pin_37)
- net PA7: now also J10.12 (Pin_12), J11.12 (Pin_12), J9.12 (Pin_12)
- net PC0: now also J10.46 (Pin_46), J11.46 (Pin_46), J9.46 (Pin_46)
- net PC1: now also J10.22 (Pin_22), J11.22 (Pin_22), J9.22 (Pin_22)
- net PC2: now also J10.47 (Pin_47), J11.47 (Pin_47), J9.47 (Pin_47)
- net PC3: now also J10.23 (Pin_23), J11.23 (Pin_23), J9.23 (Pin_23)
- net RAMA16: now also J5.66 (Pin_66), J6.66 (Pin_66), J7.66 (Pin_66), J8.66 (Pin_66)
- net RAMA17: now also J5.30 (Pin_30), J6.30 (Pin_30), J7.30 (Pin_30), J8.30 (Pin_30)
- net RAMA18: now also J5.65 (Pin_65), J6.65 (Pin_65), J7.65 (Pin_65), J8.65 (Pin_65)
- net RAMDIS: now also J1.45 (Pin_45), D26.1 (A1), J12.23 (Pin_23), J2.45 (Pin_45), J3.45 (Pin_45), J4.45 (Pin_45), J5.23 (Pin_23), J6.23 (Pin_23), J7.23 (Pin_23), J8.23 (Pin_23)
- net RD0: now also J5.71 (Pin_71), J6.71 (Pin_71), J7.71 (Pin_71), J8.71 (Pin_71)
- net RD1: now also J5.35 (Pin_35), J6.35 (Pin_35), J7.35 (Pin_35), J8.35 (Pin_35)
- net RD2: now also J5.70 (Pin_70), J6.70 (Pin_70), J7.70 (Pin_70), J8.70 (Pin_70)
- net RD3: now also J5.34 (Pin_34), J6.34 (Pin_34), J7.34 (Pin_34), J8.34 (Pin_34)
- net RD4: now also J5.69 (Pin_69), J6.69 (Pin_69), J7.69 (Pin_69), J8.69 (Pin_69)
- net RD5: now also J5.33 (Pin_33), J6.33 (Pin_33), J7.33 (Pin_33), J8.33 (Pin_33)
- net RD6: now also J5.68 (Pin_68), J6.68 (Pin_68), J7.68 (Pin_68), J8.68 (Pin_68)
- net RD7: now also J5.32 (Pin_32), J6.32 (Pin_32), J7.32 (Pin_32), J8.32 (Pin_32)
- net READY: now also J1.39 (Pin_39), D23.1 (A1), J12.20 (Pin_20), J2.39 (Pin_39), J3.39 (Pin_39), J4.39 (Pin_39), J5.20 (Pin_20), J6.20 (Pin_20), J7.20 (Pin_20), J8.20 (Pin_20)
- net RIGHT: now also J10.28 (Pin_28), J11.28 (Pin_28), J9.28 (Pin_28)
- net ROMDIS: now also J1.43 (Pin_43), D25.1 (A1), J12.22 (Pin_22), J2.43 (Pin_43), J3.43 (Pin_43), J4.43 (Pin_43)
- net SOUND: now also J1.1 (Pin_1), D4.1 (A1), J10.1 (Pin_1), J11.1 (Pin_1), J12.1 (Pin_1), J2.1 (Pin_1), J3.1 (Pin_1), J4.1 (Pin_1), J9.1 (Pin_1)
- net VSYNC: now also J10.24 (Pin_24), J11.24 (Pin_24), J5.25 (Pin_25), J6.25 (Pin_25), J7.25 (Pin_25), J8.25 (Pin_25), J9.24 (Pin_24)
- net ~244EN: now also J5.59 (Pin_59), J6.59 (Pin_59), J7.59 (Pin_59), J8.59 (Pin_59)
- net ~BRST: now also J1.40 (Pin_40), D46.1 (A1), J13.20 (Pin_20), J2.40 (Pin_40), J3.40 (Pin_40), J4.40 (Pin_40), SW2.1, U2.1 (~MR)
- net ~BUSAK: now also J1.38 (Pin_38), D45.1 (A1), J13.19 (Pin_19), J2.38 (Pin_38), J3.38 (Pin_38), J4.38 (Pin_38)
- net ~BUSRQ: now also J1.37 (Pin_37), D22.1 (A1), J12.19 (Pin_19), J2.37 (Pin_37), J3.37 (Pin_37), J4.37 (Pin_37)
- net ~CAS: now also J5.58 (Pin_58), J6.58 (Pin_58), J7.58 (Pin_58), J8.58 (Pin_58)
- net ~CPU_ADDR: now also J10.48 (Pin_48), J11.48 (Pin_48), J5.61 (Pin_61), J6.61 (Pin_61), J7.61 (Pin_61), J8.61 (Pin_61), J9.48 (Pin_48)
- net ~EXP: now also J1.48 (Pin_48), D50.1 (A1), J10.50 (Pin_50), J11.50 (Pin_50), J13.24 (Pin_24), J2.48 (Pin_48), J3.48 (Pin_48), J4.48 (Pin_48), J9.50 (Pin_50)
- net ~HALT: now also J1.34 (Pin_34), D43.1 (A1), J13.17 (Pin_17), J2.34 (Pin_34), J3.34 (Pin_34), J4.34 (Pin_34)
- net ~INT: now also J1.35 (Pin_35), D21.1 (A1), J12.18 (Pin_18), J2.35 (Pin_35), J3.35 (Pin_35), J4.35 (Pin_35), J5.19 (Pin_19), J6.19 (Pin_19), J7.19 (Pin_19), J8.19 (Pin_19)
- net ~IORQ: now also J1.31 (Pin_31), D19.1 (A1), J10.19 (Pin_19), J11.19 (Pin_19), J12.16 (Pin_16), J2.31 (Pin_31), J3.31 (Pin_31), J4.31 (Pin_31), J5.17 (Pin_17), J6.17 (Pin_17), J7.17 (Pin_17), J8.17 (Pin_17), J9.19 (Pin_19)
- net ~M1: now also J1.29 (Pin_29), D18.1 (A1), J10.18 (Pin_18), J11.18 (Pin_18), J12.15 (Pin_15), J2.29 (Pin_29), J3.29 (Pin_29), J4.29 (Pin_29), J5.16 (Pin_16), J6.16 (Pin_16), J7.16 (Pin_16), J8.16 (Pin_16), J9.18 (Pin_18)
- net ~MA0_CCLK: now also J5.57 (Pin_57), J6.57 (Pin_57), J7.57 (Pin_57), J8.57 (Pin_57)
- net ~MREQ: now also J1.28 (Pin_28), D40.1 (A1), J13.14 (Pin_14), J2.28 (Pin_28), J3.28 (Pin_28), J4.28 (Pin_28), J5.51 (Pin_51), J6.51 (Pin_51), J7.51 (Pin_51), J8.51 (Pin_51)
- net ~MWE: now also J5.63 (Pin_63), J6.63 (Pin_63), J7.63 (Pin_63), J8.63 (Pin_63)
- net ~NMI: now also J1.36 (Pin_36), D44.1 (A1), J13.18 (Pin_18), J2.36 (Pin_36), J3.36 (Pin_36), J4.36 (Pin_36)
- net ~RAMCS: now also J5.64 (Pin_64), J6.64 (Pin_64), J7.64 (Pin_64), J8.64 (Pin_64)
- net ~RAMOE: now also J5.28 (Pin_28), J6.28 (Pin_28), J7.28 (Pin_28), J8.28 (Pin_28)
- net ~RAMRD: now also J1.44 (Pin_44), D48.1 (A1), J13.22 (Pin_22), J2.44 (Pin_44), J3.44 (Pin_44), J4.44 (Pin_44), J5.54 (Pin_54), J6.54 (Pin_54), J7.54 (Pin_54), J8.54 (Pin_54)
- net ~RAMWE: now also J5.29 (Pin_29), J6.29 (Pin_29), J7.29 (Pin_29), J8.29 (Pin_29)
- net ~RAS: now also J5.62 (Pin_62), J6.62 (Pin_62), J7.62 (Pin_62), J8.62 (Pin_62)
- net ~RD: now also J1.32 (Pin_32), D42.1 (A1), J10.42 (Pin_42), J11.42 (Pin_42), J13.16 (Pin_16), J2.32 (Pin_32), J3.32 (Pin_32), J4.32 (Pin_32), J5.52 (Pin_52), J6.52 (Pin_52), J7.52 (Pin_52), J8.52 (Pin_52), J9.42 (Pin_42)
- net ~RFSH: now also J1.30 (Pin_30), D41.1 (A1), J13.15 (Pin_15), J2.30 (Pin_30), J3.30 (Pin_30), J4.30 (Pin_30)
- net ~ROMEN: now also J1.42 (Pin_42), D47.1 (A1), J13.21 (Pin_21), J2.42 (Pin_42), J3.42 (Pin_42), J4.42 (Pin_42), J5.53 (Pin_53), J6.53 (Pin_53), J7.53 (Pin_53), J8.53 (Pin_53)
- net ~RSET: now also J1.41 (Pin_41), D24.1 (A1), J10.21 (Pin_21), J11.21 (Pin_21), J12.21 (Pin_21), J2.41 (Pin_41), J3.41 (Pin_41), J4.41 (Pin_41), J5.21 (Pin_21), J6.21 (Pin_21), J7.21 (Pin_21), J8.21 (Pin_21), J9.21 (Pin_21), U2.7 (~RESET)
- net ~WR: now also J1.33 (Pin_33), D20.1 (A1), J10.20 (Pin_20), J11.20 (Pin_20), J12.17 (Pin_17), J2.33 (Pin_33), J3.33 (Pin_33), J4.33 (Pin_33), J5.18 (Pin_18), J6.18 (Pin_18), J7.18 (Pin_18), J8.18 (Pin_18), J9.20 (Pin_20)
- net +5V: now reaches J1.27 (Pin_27)
- net +5V: now also C2.1, C4.1, D17.1 (A1), D2.1 (A1), J10.17 (Pin_17), J11.17 (Pin_17), J12.14 (Pin_14), J15.1 (Pin_1), J17.2 (Pin_2), J2.27 (Pin_27), J3.27 (Pin_27), J4.27 (Pin_27), J5.15 (Pin_15), J6.15 (Pin_15), J7.15 (Pin_15), J8.15 (Pin_15), J9.17 (Pin_17), R1.1, U1.6 (Vout+), U2.2 (Vcc)
- new net: D3.2 (A), R1.2
- new net: D1.1 (A1), F1.1, TH1.2
- new net: SW1.2 (B), TH1.1
- new net +12V: C3.1, D53.1 (A1), J15.4 (Pin_4), U3.4 (+VOUT)
- new net A14OUT: J5.38 (Pin_38), J6.38 (Pin_38), J7.38 (Pin_38), J8.38 (Pin_38)
- new net A15OUT: J5.2 (Pin_2), J6.2 (Pin_2), J7.2 (Pin_2), J8.2 (Pin_2)
- new net PLUS: J14.3 (D+)
- new net PRTBSY: J10.49 (Pin_49), J11.49 (Pin_49), J9.49 (Pin_49)
- new net SPARE1: J5.1 (Pin_1), J6.1 (Pin_1), J7.1 (Pin_1), J8.1 (Pin_1)
- new net SPARE2: J5.22 (Pin_22), J6.22 (Pin_22), J7.22 (Pin_22), J8.22 (Pin_22)
- new net SPARE3: J5.31 (Pin_31), J6.31 (Pin_31), J7.31 (Pin_31), J8.31 (Pin_31)
- new net SPARE4: J5.67 (Pin_67), J6.67 (Pin_67), J7.67 (Pin_67), J8.67 (Pin_67)
- new net SPARE5: J5.72 (Pin_72), J6.72 (Pin_72), J7.72 (Pin_72), J8.72 (Pin_72)
- new net SWITCHED_5V: C1.1, SW1.1 (A), U1.2 (Vin+), U2.4 (PFI), U3.2 (+VIN)
- new net UGND: C1.2, D1.2 (A2), J14.4 (GND), J14.5 (Shield), U1.1 (Vin-)
- new net VBUS: F1.2, J14.1 (VBUS)
- new net ~XCPU_AD: J5.60 (Pin_60), J6.60 (Pin_60), J7.60 (Pin_60), J8.60 (Pin_60)
- no-connect marks 0 -> 9
Other:
- note added: "Attach a lead and 2.1mm phono plug to the power out.\nCan be used to power a CPC to SCART lead. \nSocket can be used for safe storage of the plug.\nPlug should be wired centre-positive."
- note added: "DISC POWER OUT"
- note added: "ESD PROTECTION FOR EXPANSION CONNECTOR"
- note added: "Expansion\n(Edge connector)"
- note added: "POWER IN"
- note added: "RESET"
- note added: "SCART POWER AND\nJACK STORAGE"
- note removed: "SPARE but connected"
- moved on the sheet: J1
