File: DDI20/CPC-DDI20.kicad_pcb (KiCad board)
At the start: 2 copper layers, 99.1 x 49.9 mm, 47 parts, among them IC201 UPD765AC, IC202 FDC9229, IC203 74LS04, IC205 74LS08, IC206 74LS38, IC207 74LS32, IC208 74LS38, IC209 74LS86, IC210 74LS132, IC212 74LS74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

Commit message: Long overdue update...
Parts:
- removed C10, C9: 0.1nF, Capacitor_THT:C_Disc_D3.0mm_W2.0mm_P2.50mm
- removed J1: RC2014Bus, Connector_PinHeader_2.54mm:PinHeader_1x40_P2.54mm_Vertical
- removed JP1: DS Type, Connector_PinHeader_2.54mm:PinHeader_1x03_P2.54mm_Vertical
- removed NR201-1, NR201-3, NR201-4, NR201-5, NR201-7: 680R, Resistor_THT:R_Axial_DIN0207_L6.3mm_D2.5mm_P7.62mm_Horizontal
- added J2: MX4 Connector, Connector_IDC:IDC-Header_2x25_P2.54mm_Horizontal, F.Cu at (219.7, 161.9)
- added RN201: 680, Resistor_THT:R_Array_SIP6, F.Cu at (228.6, 111.8)
- C102: value 47P (NPO) -> 47p (NPO); footprint Capacitor_THT:C_Radial_D5.0mm_H5.0mm_P2.00mm -> Capacitor_THT:C_Disc_D3.0mm_W2.0mm_P2.50mm
- J3: value Conn_02x17_Odd_Even -> Channel 1
- J4: value Conn_02x17_Odd_Even -> Channel 2
- SW1: value A/B Switch -> ABBA; footprint Button_Switch_THT:SW_E-Switch_EG1271_DPDT -> Button_Switch_THT:SW_CuK_OS102011MA1QN1_SPDT_Angled
- moved J4 67.3 mm to (246.4, 118.1), turned to 0 degrees
- moved NR201-6 52.6 mm to (156.8, 123.8)
- moved SW1 48.5 mm to (242.6, 106.7), turned to 180 degrees
- moved IC201 44.3 mm to (182.9, 106.0), turned to 0 degrees
- moved C5 33.5 mm to (205.7, 117.5)
- moved C6 33.0 mm to (205.1, 106.7)
- moved IC208 31.1 mm to (213.4, 135.9)
- moved IC205 30.5 mm to (160.7, 123.8)
- moved J3 30.1 mm to (236.2, 118.1), turned to 0 degrees
- moved R212 29.8 mm to (179.7, 141.6), turned to 270 degrees
- moved IC202 28.9 mm to (201.3, 131.4), turned to 0 degrees
- moved R109 28.7 mm to (220.3, 142.2), turned to 180 degrees
- moved Q101 28.7 mm to (218.4, 154.3), turned to 90 degrees
- moved IC206 28.3 mm to (208.9, 114.3)
- moved R113 24.1 mm to (156.8, 150.5), turned to 270 degrees
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Connections:
- net Net-(IC201-Pad15) renamed /DDI/5V_PUP
- IC203 pad 12: /DDI/DDI-FDDS/~DSKD -> Net-(IC201-Pad35)
- IC203 pad 13: /DDI/~READ_DATA -> /DDI/~READY
- IC203 pad 3: /DDI/~READY -> /DDI/~TRACK0
- IC203 pad 4: Net-(IC201-Pad35) -> Net-(IC203-Pad4)
- IC203 pad 5: /DDI/~TRACK0 -> /DDI/~INDEX
- IC203 pad 6: Net-(IC203-Pad6) -> Net-(IC201-Pad17)
- IC203 pad 8: Net-(IC201-Pad17) -> /DDI/DDI-FDDS/~DSKD
- IC203 pad 9: /DDI/~INDEX -> /DDI/~READ_DATA
- IC205 pad 12: Net-(IC205-Pad12) -> /DDI/DEVICE_SELECT
- IC205 pad 13: /DDI/DEVICE_SELECT -> Net-(IC205-Pad13)
- IC205 pad 2: /DDI/CLK4 -> /CLK4
- IC205 pad 5: Net-(IC203-Pad6) -> Net-(IC203-Pad4)
- IC206 pad 10: Net-(IC201-Pad29) -> Net-(IC206-Pad10)
- IC206 pad 11: Net-(IC206-Pad11) -> /DDI/~DRIVE_SELECT_1
- IC206 pad 12: Net-(IC206-Pad12) -> /DDI/~DRIVE_SELECT_0
- IC206 pad 13: Net-(IC206-Pad12) -> /DDI/~DRIVE_SELECT_0
- IC206 pad 8: Net-(IC206-Pad8) -> /DDI/~DRIVE_SELECT_0
- IC206 pad 9: Net-(IC201-Pad29) -> Net-(IC206-Pad10)
- IC207 pad 10: /DDI/~RD -> /~IORQ
- IC207 pad 4: /DDI/~WR -> /~RD
- IC207 pad 5: /DDI/IORQ -> /~IORQ
- IC207 pad 6: Net-(IC201-Pad3) -> Net-(IC201-Pad2)
- IC207 pad 8: Net-(IC201-Pad2) -> Net-(IC201-Pad3)
- IC207 pad 9: /DDI/IORQ -> /~WR
- IC208 pad 10: Net-(IC205-Pad8) -> /DDI/DDI-FDDS/WDOUT
- IC208 pad 4: /DDI/DDI-FDDS/WDOUT -> Net-(IC205-Pad8)
- IC208 pad 5: /DDI/DDI-FDDS/WDOUT -> Net-(IC205-Pad8)
- IC208 pad 6: /DDI/~WRITE_DATA -> /DDI/~STEP
- IC208 pad 8: /DDI/~STEP -> /DDI/~WRITE_DATA
- IC208 pad 9: Net-(IC205-Pad8) -> /DDI/DDI-FDDS/WDOUT
- IC209 pad 10: +5V -> Net-(IC209-Pad10)
- IC209 pad 3: Net-(IC205-Pad12) -> Net-(IC205-Pad13)
- IC209 pad 8: Net-(IC209-Pad8) -> Net-(IC206-Pad10)
- IC209 pad 9: +5V -> Net-(IC201-Pad29)
- R118 pad 1: /DDI/~RESET -> /~RESET
- R214 pad 1: Net-(IC206-Pad12) -> /DDI/~DRIVE_SELECT_0
- SW1 pad 1: /DDI/~DRIVE_SELECT_0 -> GND
- SW1 pad 2: Net-(IC206-Pad11) -> Net-(IC209-Pad10)
- SW1 pad 3: /DDI/~DRIVE_SELECT_1 -> +5V
Routing:
- net Net-(IC209-Pad10): track 0.00 -> 99.1 mm, vias 0 -> 1
- net /CLK4: track 0.00 -> 89.3 mm, vias 0 -> 2
- net /DDI/DDI-FDDS/CLK_4: track 96.7 -> 18.1 mm, vias 2 -> 0
- net Net-(IC206-Pad10): track 0.00 -> 67.2 mm, vias 0 -> 1
- net +5V: track 379.2 -> 317.7 mm
- net /DDI/IORQ: track 60.7 -> 0.00 mm
- net Net-(IC201-Pad28): track 57.4 -> 0.00 mm, vias 1 -> 0
- net /DDI/~RD: track 55.1 -> 0.00 mm, vias 1 -> 0
- net GND: track 528.5 -> 477.3 mm
- net Net-(IC203-Pad6): track 49.3 -> 0.00 mm, vias 2 -> 0
- net /DDI/~WR: track 48.8 -> 0.00 mm
- net Net-(IC203-Pad4): track 0.00 -> 47.4 mm
- net Net-(IC205-Pad8): track 14.4 -> 60.0 mm, vias 0 -> 1
- net /DDI/5V_PUP: track 96.2 -> 50.9 mm, vias 2 -> 0
- net D1: track 9.43 -> 50.0 mm
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- added copper zone on B.Cu, net GND
- added copper zone on F.Cu, net GND
Other:
- board size 99.1 x 49.9 mm -> 99.1 x 65.9 mm
- rule pad_to_mask_clearance: 0.2 -> 0
- board text added: "ABBA switch swaps drive designations on both channels. Ie. drives will be swapped whether both on one channel or on separate channels. Channels: * Both drives on one channel (1) configured as A and B (via drive or cable). * One drive on each channel with both drives configured as A."
- board text added: "All capacitors are 0.1uF unless marked. C102 states NPO, which probably means non-polarized. IC209 *must* be 74LS86. Do not substitute other logic series."
- board text added: "CPC Floppy Controller"
- board text added: "Floppy disc controller for Amstrad CPC © Mike Sutton - Bread80.com mstdn.com/bread80 - github.com/bread80"
- board text added: "MX4"
- board text added: "NORMAL"
- board text added: "REV 1"
- board text added: "SWAP"
- board text removed: "Pin 1"
