File: DDI20/CPC-DDI20.sch (KiCad schematic (older format))
At the start: 11 parts, among them J1 RC2014Bus

Commit message: Long overdue update...
Parts:
- removed C10, C9: 0.1nF, Capacitor_THT:C_Disc_D3.0mm_W2.0mm_P2.50mm, symbol Device:C
- removed J1: RC2014Bus, Connector_PinHeader_2.54mm:PinHeader_1x40_P2.54mm_Vertical, symbol CPC:RC2014Bus
- added J2: MX4 Connector, Connector_IDC:IDC-Header_2x25_P2.54mm_Horizontal, symbol Connector_Generic:Conn_02x25_Odd_Even
Connections:
- net +5V: now also J2.24 (Pin_24)
- net A0: now also J2.33 (Pin_33)
- net A10: now also J2.43 (Pin_43)
- net A7: now also J2.40 (Pin_40)
- net A8: now also J2.41 (Pin_41)
- net D0: now also J2.25 (Pin_25)
- net D1: now also J2.26 (Pin_26)
- net D2: now also J2.27 (Pin_27)
- net D3: now also J2.28 (Pin_28)
- net D4: now also J2.29 (Pin_29)
- net D5: now also J2.30 (Pin_30)
- net D6: now also J2.31 (Pin_31)
- net D7: now also J2.32 (Pin_32)
- net GND: now also J2.2 (Pin_2), J2.49 (Pin_49)
- new net CLK4: J2.1 (Pin_1)
- new net ~IORQ: J2.20 (Pin_20)
- new net ~RD: J2.19 (Pin_19)
- new net ~RESET: J2.10 (Pin_10)
- new net ~WR: J2.18 (Pin_18)
- no-connect marks 21 -> 30
