File: DDI20/DDI-FDDS.sch (KiCad schematic (older format))
At the start: 17 parts, among them IC202 FDC9229, IC209 74LS86, IC210 74LS132, Q101 2SC1815, Q102 2SC1815

Commit message: Long overdue update...
Parts:
- C102: value 47P (NPO) -> 47p (NPO); footprint Capacitor_THT:C_Radial_D5.0mm_H5.0mm_P2.00mm -> Capacitor_THT:C_Disc_D3.0mm_W2.0mm_P2.50mm
- IC202: symbol CPC:FDC9229 -> CPC-DDI20-rescue:FDC9229-CPC
Changed lines of the file:
@@
 $EndDescr
 $Comp
-L CPC:FDC9229 IC202
+L CPC-DDI20-rescue:FDC9229-CPC IC202
 U 1 1 610A1018
 P 5100 5800
+AR Path="/610A1018" Ref="IC202"  Part="1"
+AR Path="/62406B09/6109FCA9/610A1018" Ref="IC202"  Part="1"
 F 0 "IC202" H 5250 6800 50  0000 C CNN
 F 1 "FDC9229" H 5300 6700 50  0000 C CNN
@@
 P 1800 7050
 F 0 "C102" H 1915 7096 50  0000 L CNN
-F 1 "47P (NPO)" H 1915 7005 50  0000 L CNN
-F 2 "Capacitor_THT:C_Radial_D5.0mm_H5.0mm_P2.00mm" H 1838 6900 50  0001 C CNN
+F 1 "47p (NPO)" H 1915 7005 50  0000 L CNN
+F 2 "Capacitor_THT:C_Disc_D3.0mm_W2.0mm_P2.50mm" H 1838 6900 50  0001 C CNN
 F 3 "~" H 1800 7050 50  0001 C CNN
 	1    1800 7050
