File: DDI20/DDI.sch (KiCad schematic (older format))
At the start: 21 parts, among them IC201 UPD765AC, IC203 74LS04, IC205 74LS08, IC206 74LS38, IC207 74LS32, IC208 74LS38, IC209 74LS86, IC210 74LS132, IC212 74LS74, J3 Conn_02x17_Odd_Even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

Commit message: Long overdue update...
Parts:
- removed JP1: DS Type, Connector_PinHeader_2.54mm:PinHeader_1x03_P2.54mm_Vertical, symbol Jumper:Jumper_3_Bridged12
- removed NR201-1, NR201-3, NR201-4, NR201-5, NR201-7: 680R, Resistor_THT:R_Axial_DIN0207_L6.3mm_D2.5mm_P7.62mm_Horizontal, symbol Device:R
- removed SW1: A/B Switch, Button_Switch_THT:SW_E-Switch_EG1271_DPDT, symbol Switch:SW_Push_DPDT
- added RN201: 680, Resistor_THT:R_Array_SIP6, symbol Device:R_Network05
- added SW1: ABBA, Button_Switch_THT:SW_CuK_OS102011MA1QN1_SPDT_Angled, symbol Switch:SW_SPDT
- IC201: symbol CPC:UPD765AC -> CPC-DDI20-rescue:UPD765AC-CPC
- J3: value Conn_02x17_Odd_Even -> Channel 1
- J4: value Conn_02x17_Odd_Even -> Channel 2
Connections:
- net +5V: now also RN201.1 (common), SW1.3 (C); no longer IC209.10, IC209.9
- net DDI-FDDS/WDOUT: now also IC208.10, IC208.9; no longer IC208.4, IC208.5
- net DDI-FDDS/~DSKD: now also IC203.8; no longer IC203.12
- net DEVICE_SELECT: now also IC205.12; no longer IC205.13
- net GND: now also SW1.1 (A)
- net IORQ: now also IC207.10; no longer IC207.9
- net ~DRIVE_SELECT_0: now also IC206.12, IC206.13, IC206.8, R214.1
- net ~DRIVE_SELECT_1: now also IC206.11
- net ~INDEX: now also IC203.5, RN201.6 (R5); no longer IC203.9
- net ~RD: now also IC207.4; no longer IC207.10
- net ~READY: now also IC203.13, RN201.2 (R1); no longer IC203.3
- net ~READ_DATA: now also IC203.9, RN201.3 (R2); no longer IC203.13
- net ~STEP: now also IC208.6; no longer IC208.8
- net ~TRACK0: now also IC203.3, RN201.5 (R4); no longer IC203.5
- net ~WR: now also IC207.9; no longer IC207.4
- net ~WRITE_DATA: now also IC208.8; no longer IC208.6
- net ~WRITE_PROTECT: now also RN201.4 (R3)
- net at IC209.3: now also IC205.13; no longer IC205.12
- net at IC207.8: now also IC201.3 (~WR), IC207.12; no longer IC201.2 (~RD)
- net at IC206.10, IC206.9: now also IC209.8; no longer IC201.29 (US0)
- net at IC201.35 (RDY), IC208.12: now also IC203.12; no longer IC203.4
- net 5V_PUP: now reaches IC201.15 (~DACK), IC205.1, IC212.4 (~S), R212.1
- net at IC205.5: now also IC203.4; no longer IC203.6
- net at IC201.17 (IDX): now also IC203.6; no longer IC203.8
- new net: IC201.2 (~RD), IC207.6
- new net: IC205.8, IC208.4, IC208.5
- new net: IC209.10, SW1.2 (B)
- new net: IC201.29 (US0), IC209.9
Other:
- note added: "Amstrad FD1 pinout:\n(as viewed from rear)\nBottom row is GND\nTop row, left is Power pins\nTop row, right is READY"
- note added: "Connector 2: Swapped drive letters"
- note added: "NORM"
- note added: "NOTE: Amstrad connector pinouts are 'swapped'\ncompared to usual. I.e odd and even pins.\nPlug may need to be wired appropriately."
- note added: "SWAP"
- note added: "Two channels allows either:\nA and B drives on one channel, either configured via\ndrive settings or cable.\nOne drive on each channel with both drives configured as A drive.\n\nABBA switch swaps drive designations on both channels. Ie.\ndrives will be swapped whether both on one channel or on separate channels."
- note removed: "Connector 2: Reversed drive select pins. \nCan be used as B drive for a drive wired \nas A, e.g when using a floppy emulator."
- note removed: "JP1: Drive select: \nCPC vs standard"
- note removed: "SW1: A/B switch"
- moved on the sheet: IC201, IC203A, IC203B, IC203C, IC203D, IC203E, IC203F, IC203G, IC205A, IC205B, IC205C, IC205D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
