File: IO/CPCIO.sch (KiCad schematic (older format))
At the start: 6 parts, among them J902 Conn_01x08_Male

Commit message: Long overdue update...
Parts:
- removed C2: 0.1nF, Capacitor_THT:C_Disc_D3.0mm_W2.0mm_P2.50mm, symbol Device:C
- removed J902: Conn_01x08_Male, Connector_PinHeader_2.54mm:PinHeader_1x08_P2.54mm_Vertical, symbol Connector:Conn_01x08_Male
- removed JP1: RC2014Bus, Connector_PinHeader_2.54mm:PinHeader_1x40_P2.54mm_Vertical, symbol CPCIO-rescue:RC2014Bus-CPC
- removed JP2: RC2014ExtendedBus, Connector_PinHeader_2.54mm:PinHeader_1x25_P2.54mm_Vertical, symbol CPCIO-rescue:RC2014ExtendedBus-CPC
- removed LK913: Jumper_NO_Small, Connector_PinHeader_2.54mm:PinHeader_1x02_P2.54mm_Vertical, symbol Device:Jumper_NO_Small
- added JP1: CPCM_IOSound_EdgeBottom, CPCModular:Edge25_2.54PS, symbol CPCModular:CPCM_IOSound_EdgeTop
- added JP2: CPCM_IOSound_EdgeTop, CPCModular:Edge25_2.54PS, symbol CPCModular:CPCM_IOSound_EdgeBottom
Connections:
- net +5V: now also JP2.17 (Vcc)
- net A11: now also JP2.7 (A11)
- net A8: now also JP1.8 (A8)
- net A9: now also JP2.8 (A9)
- net D0: now also JP1.16 (D0)
- net D1: now also JP2.16 (D1)
- net D2: now also JP1.15 (D2)
- net D3: now also JP2.15 (D3)
- net D4: now also JP1.14 (D4)
- net D5: now also JP2.14 (D5)
- net D6: now also JP1.13 (D6)
- net D7: now also JP2.13 (D7)
- net GND: now also JP1.1 (GND), JP2.25 (GND)
- net IO_SOUND/BC1: now also JP1.19 (BC1)
- net IO_SOUND/BDIR: now also JP1.18 (BDIR)
- net IO_SOUND/VSYNC: now also JP2.24 (VSYNC)
- net IO_SOUND/~EXP: now also JP1.25 (~EXP)
- net IO_SOUND/~IORQ: now also JP2.19 (~IORQ)
- net IO_SOUND/~RD: now also JP1.17 (~RD)
- net IO_SOUND/~RESET: now also JP2.21 (~RSET)
- net IO_SOUND/~WR: now also JP2.20 (~WR)
- net PA0: now also JP1.9 (PA0)
- net PA1: now also JP2.9 (PA1)
- net PA2: now also JP1.10 (PA2)
- net PA3: now also JP2.10 (PA3)
- net PA4: now also JP1.11 (PA4)
- net PA5: now also JP2.11 (PA5)
- net PA6: now also JP1.12 (PA6)
- net PA7: now also JP2.12 (PA7)
- net PC0: now also JP1.21 (PC0)
- net PC1: now also JP2.22 (PC1)
- net PC2: now also JP1.22 (PC2)
- net PC3: now also JP2.23 (PC3)
- new net IO_SOUND/CASRD: JP2.2 (CASRD)
- new net IO_SOUND/CASWR: JP1.2 (CASWR)
- new net IO_SOUND/MOTOR: JP1.20 (MOTOR)
- new net IO_SOUND/PRTBSY: JP1.24 (PRTBSY)
- no-connect marks 19 -> 10
