File: IO/IO_SOUND.sch (KiCad schematic (older format))
At the start: 26 parts, among them IC107 8255A, J901 Conn_01x07_Male, Q101 BC337, Q901 BC337, U1 74LS688

Commit message: Long overdue update...
Parts:
- removed J901: Conn_01x07_Male, Connector_PinHeader_2.54mm:PinHeader_1x07_P2.54mm_Vertical, symbol Connector:Conn_01x07_Male
- removed JP10: A14A6, Connector_PinHeader_2.54mm:PinHeader_1x03_P2.54mm_Vertical, symbol Jumper:Jumper_3_Bridged12
- removed JP11, JP17, JP18, JP19: A10A2, Connector_PinHeader_2.54mm:PinHeader_1x03_P2.54mm_Vertical, symbol Jumper:Jumper_3_Bridged12
- removed JP12: A15A7, Connector_PinHeader_2.54mm:PinHeader_1x03_P2.54mm_Vertical, symbol Jumper:Jumper_3_Bridged12
- removed JP13, JP14, JP15, JP16, JP3, JP4, JP7, JP8: Jumper_3_Bridged12, Jumper:SolderJumper-3_P1.3mm_Open_RoundedPad1.0x1.5mm, symbol Jumper:Jumper_3_Bridged12
- removed JP5: A12A4, Connector_PinHeader_2.54mm:PinHeader_1x03_P2.54mm_Vertical, symbol Jumper:Jumper_3_Bridged12
- removed JP6: A13A5, Connector_PinHeader_2.54mm:PinHeader_1x03_P2.54mm_Vertical, symbol Jumper:Jumper_3_Bridged12
- removed JP9: A11A3, Connector_PinHeader_2.54mm:PinHeader_1x03_P2.54mm_Vertical, symbol Jumper:Jumper_3_Bridged12
- removed U1: 74LS688, Package_DIP:DIP-20_W7.62mm_Socket, symbol 74xx:74LS688
- added LK1..6: Settings, Connector_PinHeader_2.54mm:PinHeader_2x06_P2.54mm_Vertical, symbol Connector_Generic:Conn_02x06_Odd_Even
- added U901: 74LS32, Package_DIP:DIP-14_W7.62mm_Socket, symbol 74xx:74LS32
Connections:
- net A8A0 is gone; now on net A8: IC107.9 (A0)
- net A9A1 is gone; now on net A9: IC107.8 (A1)
- net +5V: now also U901.14 (VCC)
- net A11: now also U901.4
- net GND: now also LK1..6.10 (Pin_10), LK1..6.12 (Pin_12), LK1..6.2 (Pin_2), LK1..6.4 (Pin_4), LK1..6.6 (Pin_6), LK1..6.8 (Pin_8), U901.1, U901.10, U901.12, U901.13, U901.2, U901.7 (GND), U901.9
- net PRTBSY: now also LK1..6.1 (Pin_1)
- net REG0: now also LK1..6.11 (Pin_11)
- net REG1: now also LK1..6.9 (Pin_9)
- net REG2: now also LK1..6.7 (Pin_7)
- net Tape/~MOTORINT: now also Q101.1 (C)
- net VIDFRQ: now also LK1..6.5 (Pin_5)
- net ~EXP: now also LK1..6.3 (Pin_3)
- net ~IORQ: now also U901.5
- net MOTOR: now reaches IC107.13 (PC4), R113.1
- net at IC107.6 (~CS~): now also U901.6
- net RD_DATA renamed CASRD
- net WR_DATA renamed CASWR
- no-connect marks 0 -> 3
Other:
- note removed: "For CPC: A11 low, all others high."
- note removed: "Set jumpers to '1' for CPC (high byte of IO address)\nto '3' for RC2014 (low byyte of IO address)."
- moved on the sheet: Q101, R113
