File: IO/Tape.sch (KiCad schematic (older format))
At the start: 25 parts, among them IC301 LM358, J1 Tape in, J2 Tape out, J3 Motor

Commit message: Long overdue update...
Parts:
- J3: footprint Connector_Audio:Jack_3.5mm_CUI_SJ1-3533NG_Horizontal -> CPCModular:CUI_MJ1_2503A
Connections:
- net CASRDINT: now also IC301.1; no longer IC301.7
- net GNDA: now also IC301.5 (+); no longer IC301.3 (+)
- net at C318.1, RY30.3: now also J3.T; no longer J3.S
- net at C318.2, RY30.2: now also J3.S; no longer J3.T
- net at C314.1, D301.2 (A), D302.1 (K)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: now also IC301.3 (+); no longer IC301.5 (+)
- net at C315.1, R307.1, R311.1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: now also IC301.2 (-); no longer IC301.6 (-)
- new net: IC301.6 (-), IC301.7
Other:
- note added: "2.5mm audio jack,\nE.g. CUI MJ1-2503A"
- note added: "3.5mm Sockets are CUI \nSJ1-3533NG"
- note removed: "Sockets are CUI \nSJ1-3533NG"
- moved on the sheet: J3
Changed lines of the file:
@@
 L Connector:AudioJack2 J3
 U 1 1 6369C542
-P 6800 4350
-F 0 "J3" H 6620 4425 50  0000 R CNN
-F 1 "Motor" H 6620 4334 50  0000 R CNN
-F 2 "Connector_Audio:Jack_3.5mm_CUI_SJ1-3533NG_Horizontal" H 6800 4350 50  0001 C CNN
-F 3 "~" H 6800 4350 50  0001 C CNN
-	1    6800 4350
-	-1   0    0    -1
+P 6800 4250
+F 0 "J3" H 6620 4325 50  0000 R CNN
+F 1 "Motor" H 6620 4234 50  0000 R CNN
+F 2 "CPCModular:CUI_MJ1_2503A" H 6800 4250 50  0001 C CNN
+F 3 "https://www.mouser.co.uk/datasheet/2/670/mj1_2503a-1778180.pdf" H 6800 4250 50  0001 C CNN
+	1    6800 4250
+	-1   0    0    1
 $EndComp
 $Comp
@@
 $Comp
 L Amplifier_Operational:LM358 IC301
-U 2 1 636A9894
+U 1 1 636A9894
 P 4300 3000
 F 0 "IC301" H 4300 3367 50  0000 C CNN
@@
 F 2 "Package_DIP:DIP-8_W7.62mm_Socket" H 4300 3000 50  0001 C CNN
 F 3 "http://www.ti.com/lit/ds/symlink/lm2904-n.pdf" H 4300 3000 50  0001 C CNN
-	2    4300 3000
+	1    4300 3000
 	1    0    0    -1
 $EndComp
@@
 P 3250 3400
 F 0 "#PWR0121" H 3250 3150 50  0001 C CNN
-F 1 "GNDA" H 3255 3227 50  0000 C CNN
+F 1 "GNDA" H 3150 3250 50  0000 C CNN
 F 2 "" H 3250 3400 50  0001 C CNN
 F 3 "" H 3250 3400 50  0001 C CNN
@@
 $Comp
 L Amplifier_Operational:LM358 IC301
-U 1 1 63D68FDC
+U 2 1 63D68FDC
 P 3500 5950
 F 0 "IC301" H 3500 6317 50  0000 C CNN
@@
 F 2 "Package_DIP:DIP-8_W7.62mm_Socket" H 3500 5950 50  0001 C CNN
 F 3 "http://www.ti.com/lit/ds/symlink/lm2904-n.pdf" H 3500 5950 50  0001 C CNN
-	1    3500 5950
+	2    3500 5950
 	1    0    0    -1
 $EndComp
@@
 	3100 6050 3200 6050
 $Comp
-L power:GNDA #PWR?
+L power:GNDA #PWR0103
 U 1 1 63D6CBB8
 P 3100 5850
-F 0 "#PWR?" H 3100 5600 50  0001 C CNN
+F 0 "#PWR0103" H 3100 5600 50  0001 C CNN
 F 1 "GNDA" H 3000 5850 50  0000 C CNN
 F 2 "" H 3100 5850 50  0001 C CNN
@@
 	3100 5850 3200 5850
 $Comp
-L power:+5VA #PWR?
+L power:+5VA #PWR0130
 U 1 1 63D78E38
 P 2700 1050
-F 0 "#PWR?" H 2700 900 50  0001 C CNN
+F 0 "#PWR0130" H 2700 900 50  0001 C CNN
 F 1 "+5VA" H 2715 1223 50  0000 C CNN
 F 2 "" H 2700 1050 50  0001 C CNN
@@
 $EndComp
 $Comp
-L power:+5VA #PWR?
+L power:+5VA #PWR0131
 U 1 1 63D797A6
 P 2900 2300
-F 0 "#PWR?" H 2900 2150 50  0001 C CNN
+F 0 "#PWR0131" H 2900 2150 50  0001 C CNN
 F 1 "+5VA" H 2915 2473 50  0000 C CNN
 F 2 "" H 2900 2300 50  0001 C CNN
@@
 	2900 2300 2900 2400
 $Comp
-L power:+5VA #PWR?
+L power:+5VA #PWR0132
 U 1 1 63D7DD58
 P 4250 5550
-F 0 "#PWR?" H 4250 5400 50  0001 C CNN
+F 0 "#PWR0132" H 4250 5400 50  0001 C CNN
 F 1 "+5VA" H 4265 5723 50  0000 C CNN
 F 2 "" H 4250 5550 50  0001 C CNN
@@
 $EndComp
 $Comp
-L power:+5VA #PWR?
+L power:+5VA #PWR0133
 U 1 1 63D7E655
 P 5250 1150
-F 0 "#PWR?" H 5250 1000 50  0001 C CNN
+F 0 "#PWR0133" H 5250 1000 50  0001 C CNN
 F 1 "+5VA" H 5265 1323 50  0000 C CNN
 F 2 "" H 5250 1150 50  0001 C CNN
@@
 	2600 1150 2700 1150
 Text Notes 6650 2700 0    50   ~ 0
-Sockets are CUI \nSJ1-3533NG
+3.5mm Sockets are CUI \nSJ1-3533NG
+Text Notes 6750 4050 0    50   ~ 0
+2.5mm audio jack,\nE.g. CUI MJ1-2503A
 $EndSCHEMATC
