File: RAM/CRTC_ADDR_MULTI.sch (KiCad schematic (older format))
At the start: 8 parts, among them IC108 MC6845, IC110 74LS00, IC201 74LS157, IC202 74LS157, IC203 74LS157, IC204 74LS157, U191 AS6C4008-55PCN

Commit message: Long overdue update...
Connections:
- net A14OUT is gone; now on net RAMA14: IC204.2 (I0a)
- net A15OUT is gone; now on net RAMA15: IC203.2 (I0a)
- net RAMA11: now also U191.25 (A11); no longer U191.11 (A1)
- net RAMA14: now also U191.26 (A9); no longer U191.12 (A0)
- net RAMA16: now also U191.12 (A0); no longer U191.26 (A9)
- net RAMA17: now also U191.11 (A1); no longer U191.25 (A11)
- net RAMA18: now also U191.10 (A2); no longer U191.23 (A10)
- net RAMA7: now also U191.23 (A10); no longer U191.10 (A2)
- net at IC110.10: now also IC110.3; no longer IC110.6
- net at IC110.9: now also IC110.6; no longer IC110.3
- net RAMD0 renamed RD7
- net RAMD1 renamed RD6
- net RAMD2 renamed RD4
- net RAMD3 renamed RD2
- net RAMD4 renamed RD0
- net RAMD5 renamed RD5
- net RAMD6 renamed RD3
- net RAMD7 renamed RD1
Changed lines of the file:
@@
 F 3 "http://www.ti.com/lit/gpn/sn74ls00" H 1050 3900 50  0001 C CNN
 	3    1050 3900
-	0    -1   -1   0
+	0    1    -1   0
 $EndComp
 Wire Wire Line
@@
 Text Label 9000 4600 0    50   ~ 0
 RAMA5
-Text Label 9000 4300 0    50   ~ 0
+Text Label 9000 5100 0    50   ~ 0
 RAMA7
 Text Label 9000 5700 0    50   ~ 0
@@
 Text Label 9000 5500 0    50   ~ 0
 RAMA10
-Text Label 9000 4200 0    50   ~ 0
+Text Label 9000 5200 0    50   ~ 0
 RAMA11
 Text Label 9000 4900 0    50   ~ 0
 RAMA12
-Text Label 9000 4100 0    50   ~ 0
+Text Label 9000 5000 0    50   ~ 0
 RAMA14
 Text Label 9000 4800 0    50   ~ 0
@@
 Text Label 9000 5300 0    50   ~ 0
 RAMA15
-Text Label 9000 5000 0    50   ~ 0
+Text Label 9000 4100 0    50   ~ 0
 RAMA16
 $Comp
@@
 	1    0    0    -1
 $EndComp
-Text Label 10350 4800 0    50   ~ 0
-RAMD0
-Text Label 10350 4700 0    50   ~ 0
-RAMD1
-Text Label 10350 4600 0    50   ~ 0
-RAMD2
-Text Label 10350 4500 0    50   ~ 0
-RAMD3
-Text Label 10350 4400 0    50   ~ 0
-RAMD4
-Text Label 10350 4100 0    50   ~ 0
-RAMD5
-Text Label 10350 4200 0    50   ~ 0
-RAMD6
-Text Label 10350 4300 0    50   ~ 0
-RAMD7
+Text Label 10450 4400 0    50   ~ 0
+RD0
+Text Label 10450 4300 0    50   ~ 0
+RD1
+Text Label 10450 4500 0    50   ~ 0
+RD2
+Text Label 10450 4200 0    50   ~ 0
+RD3
+Text Label 10450 4600 0    50   ~ 0
+RD4
+Text Label 10450 4100 0    50   ~ 0
+RD5
+Text Label 10450 4700 0    50   ~ 0
+RD6
+Text Label 10450 4800 0    50   ~ 0
+RD7
 Wire Wire Line
 	10600 4100 10350 4100
@@
 	9350 5700 9000 5700
 Text GLabel 10700 3950 2    50   BiDi ~ 0
-RAMD[0..7]
+RD[0..7]
 Text HLabel 10700 3850 1    50   BiDi ~ 0
 RAMD
@@
 RAMA16
 Text HLabel 3050 5050 0    50   Input ~ 0
-A15OUT
+RAMA15
 Text HLabel 3050 5750 0    50   Input ~ 0
-A14OUT
+RAMA14
 Wire Wire Line
 	3050 5050 4200 5050
@@
 Wire Wire Line
 	9000 5900 9350 5900
-Text Label 9000 5200 0    50   ~ 0
+Text Label 9000 4200 0    50   ~ 0
 RAMA17
-Text Label 9000 5100 0    50   ~ 0
+Text Label 9000 4300 0    50   ~ 0
 RAMA18
 $Comp
