File: RAMControl/CPCRAMCtrl.sch (KiCad schematic (older format))
At the start: 13 parts, among them J1 Conn_01x10_Female, J2 Conn_01x16_Female

Commit message: Long overdue update...
Parts:
- removed J1: Conn_01x10_Female, Connector_PinSocket_2.54mm:PinSocket_1x10_P2.54mm_Vertical, symbol Connector:Conn_01x10_Female
- removed J2: Conn_01x16_Female, Connector_PinHeader_2.54mm:PinHeader_2x08_P2.54mm_Vertical, symbol Connector:Conn_01x16_Female
- removed JP1: RC2014Bus, Connector_PinHeader_2.54mm:PinHeader_1x40_P2.54mm_Vertical, symbol CPCRAMCtrl-rescue:RC2014Bus-CPC
- removed JP2: RC2014ExtendedBus, Connector_PinHeader_2.54mm:PinHeader_1x25_P2.54mm_Vertical, symbol CPCRAMCtrl-rescue:RC2014ExtendedBus-CPC
- added JP1: CPCM_VideoRAM_EdgeBottom, CPCModular:Edge36_2.54PS, symbol CPCModular:CPCM_VideoRAM_EdgeBottom
- added JP2: CPCM_VideoRAM_EdgeTop, CPCModular:Edge36_2.54PS, symbol CPCModular:CPCM_VideoRAM_EdgeTop
Connections:
- net +5V: now also JP2.15 (Vcc)
- net A14: now also JP1.3 (A14)
- net A15: now also JP2.3 (A15)
- net CRTC_ADDR_MULTI/RAMA16: now also JP1.30 (RAMA16)
- net CRTC_ADDR_MULTI/RAMA17: now also JP2.30 (RAMA17)
- net CRTC_ADDR_MULTI/RAMA18: now also JP1.29 (RAMA18)
- net CRTC_ADDR_MULTI/~244EN: now also JP1.23 (~244EN)
- net CRTC_ADDR_MULTI/~CAS: now also JP1.22 (~CAS)
- net CRTC_ADDR_MULTI/~IORQ: now also JP2.17 (~IORQ)
- net CRTC_ADDR_MULTI/~MWE: now also JP1.27 (~MWE)
- net CRTC_ADDR_MULTI/~RAMCS: now also JP1.28 (~RAMCS)
- net CRTC_ADDR_MULTI/~RAMOE: now also JP2.28 (~RAMOE)
- net CRTC_ADDR_MULTI/~RAMWE: now also JP2.29 (~RAMWE)
- net CRTC_ADDR_MULTI/~RAS: now also JP1.26 (~RAS)
- net CRTC_ADDR_MULTI/~RESET: now also JP2.21 (~RSET)
- net CRTC_ADDR_MULTI/~WR: now also JP2.18 (~WR)
- net CRTC_ADDR_MULTI/~XCPU_AD: now also JP1.24 (~XCPU_AD)
- net D0: now also JP1.14 (D0)
- net D1: now also JP2.14 (D1)
- net D2: now also JP1.13 (D2)
- net D3: now also JP2.13 (D3)
- net D4: now also JP1.12 (D4)
- net D5: now also JP2.12 (D5)
- net D6: now also JP1.11 (D6)
- net D7: now also JP2.11 (D7)
- net GND: now also JP1.1 (GND), JP2.36 (GND)
- net RAMDIS: now also JP2.23 (RAMDIS)
- net READY: now also JP2.20 (READY)
- net ~CPU_ADDR: now also JP1.25 (~CPU_ADDR)
- net ~RAMRD: now also JP1.18 (~RAMRD)
- new net CRTC_ADDR_MULTI/AOUT14: JP1.2 (A14OUT)
- new net CRTC_ADDR_MULTI/AOUT15: JP2.2 (A15OUT)
- new net RD0: JP1.35 (RD0)
- new net RD1: JP2.35 (RD1)
- new net RD2: JP1.34 (RD2)
- new net RD3: JP2.34 (RD3)
- new net RD4: JP1.33 (RD4)
- new net RD5: JP2.33 (RD5)
- new net RD6: JP1.32 (RD6)
- new net RD7: JP2.32 (RD7)
- no-connect marks 35 -> 31
Other:
- note removed: "To RAM board"
- note removed: "To video board"
