File: RAMControl/CRTC_ADDR_MULTI.sch (KiCad schematic (older format))
At the start: 17 parts, among them IC112 74LS32, IC118 AMG40031, IC192 74LS32, U114 74LS373, U115 74LS244, U191 74LS04, U193 74LS08, U194 74LS173, U195 74LS74

Commit message: Added image to readme
Parts:
- removed unit 4 of IC192
- added U192: 74LS32, Package_DIP:DIP-14_W7.62mm_Socket, symbol 74xx:74LS32
Connections:
- net GND: now also U191.13, U192.12, U192.13
- net ~244EN: no longer U191.13
- net ~CAS: no longer IC192.1
- net ~XCPU_AD: now also IC192.1
- net XCPU_AD: now reaches U195.8 (~Q)
- net XCPU_AD: now also U193.1
- net ~CPU_ADDRx renamed ~BUF_CPU_AD
- no-connect marks 7 -> 8
Other:
- note added: "Buffer ~CPU_ADDR~ for signal\nintegrity reasons"
- note added: "EXPANSION RAM CONTROL"
- note added: "Ensure ~RAMOE~ doesn't clash with ~RAMWE~.\nDuring CPU cycles, only allow RAM to output (~RAMOE~) when\n~RAMRD~ is active. During video cycles hold ~RAMOE~ active.\nRAM reads will be enabled or disabled by ~RAMCS~.\nThis could be improved but it works."
- note removed: "Allow RAM output during video cycles via ~CAS~.\nDuring CPU cycles guard against clashes with ~MWE~."
- note removed: "EXP RAM CONTROL"
- moved on the sheet: IC112B, IC192A, U193A
Changed lines of the file:
@@
 L 74xx:74LS32 IC112
 U 2 1 60FA7135
-P 2900 2150
-F 0 "IC112" H 3050 2450 50  0000 C CNN
-F 1 "74LS32" H 3050 2350 50  0000 C CNN
-F 2 "Package_DIP:DIP-14_W7.62mm_Socket" H 2900 2150 50  0001 C CNN
-F 3 "http://www.ti.com/lit/gpn/sn74ls00" H 2900 2150 50  0001 C CNN
-	2    2900 2150
+P 3050 2250
+F 0 "IC112" H 3200 2550 50  0000 C CNN
+F 1 "74LS32" H 3200 2450 50  0000 C CNN
+F 2 "Package_DIP:DIP-14_W7.62mm_Socket" H 3050 2250 50  0001 C CNN
+F 3 "http://www.ti.com/lit/gpn/sn74ls00" H 3050 2250 50  0001 C CNN
+	2    3050 2250
 	1    0    0    -1
 $EndComp
@@
 Wire Wire Line
 	3600 1300 3700 1300
-Wire Wire Line
-	3700 1100 3600 1100
 Text Notes 9150 1350 0    100  ~ 0
 BUS CONTROL
@@
 Text HLabel 950  1300 0    50   Input ~ 0
 ~RAS
-Wire Wire Line
-	950  900  1700 900
 Wire Wire Line
 	1700 900  1700 1200
@@
 Wire Wire Line
 	2450 1200 2550 1200
-NoConn ~ 2450 1400
 Text Notes 1450 750  0    50   ~ 0
 Delay multiplexers until \nafter memory writes
@@
 Wire Wire Line
 	4300 1500 4300 1400
-Text HLabel 8300 1600 2    50   Output ~ 0
+Text HLabel 8000 1600 2    50   Output ~ 0
 ~RAMOE
 $Comp
 L 74xx:74LS08 U193
 U 1 1 6395DF31
-P 7900 1600
-F 0 "U193" H 7900 1925 50  0000 C CNN
-F 1 "74LS08" H 7900 1834 50  0000 C CNN
-F 2 "Package_DIP:DIP-14_W7.62mm_Socket" H 7900 1600 50  0001 C CNN
-F 3 "http://www.ti.com/lit/gpn/sn74LS04" H 7900 1600 50  0001 C CNN
-	1    7900 1600
-	1    0    0    -1
-$EndComp
-$Comp
-L 74xx:74LS32 IC192
-U 4 1 6395F251
-P 7100 1350
-F 0 "IC192" H 7100 1675 50  0000 C CNN
-F 1 "74LS32" H 7100 1584 50  0000 C CNN
-F 2 "Package_DIP:DIP-14_W7.62mm_Socket" H 7100 1350 50  0001 C CNN
-F 3 "http://www.ti.com/lit/gpn/sn74LS32" H 7100 1350 50  0001 C CNN
-	4    7100 1350
+P 7600 1600
+F 0 "U193" H 7600 1925 50  0000 C CNN
+F 1 "74LS08" H 7600 1834 50  0000 C CNN
+F 2 "Package_DIP:DIP-14_W7.62mm_Socket" H 7600 1600 50  0001 C CNN
+F 3 "http://www.ti.com/lit/gpn/sn74LS04" H 7600 1600 50  0001 C CNN
+	1    7600 1600
 	1    0    0    -1
 $EndComp
@@
 L 74xx:74LS32 IC192
 U 1 1 63960994
-P 7100 1850
-F 0 "IC192" H 7100 2175 50  0000 C CNN
-F 1 "74LS32" H 7100 2084 50  0000 C CNN
-F 2 "Package_DIP:DIP-14_W7.62mm_Socket" H 7100 1850 50  0001 C CNN
-F 3 "http://www.ti.com/lit/gpn/sn74LS32" H 7100 1850 50  0001 C CNN
-	1    7100 1850
+P 6800 1850
+F 0 "IC192" H 6800 2175 50  0000 C CNN
+F 1 "74LS32" H 6800 2084 50  0000 C CNN
+F 2 "Package_DIP:DIP-14_W7.62mm_Socket" H 6800 1850 50  0001 C CNN
+F 3 "http://www.ti.com/lit/gpn/sn74LS32" H 6800 1850 50  0001 C CNN
+	1    6800 1850
 	1    0    0    -1
 $EndComp
@@
 	1    0    0    -1
 $EndComp
-Text HLabel 6000 1250 0    50   Input ~ 0
-~244EN
-Text HLabel 6000 1600 0    50   Input ~ 0
-~CAS
-Text HLabel 6000 1950 0    50   Input ~ 0
+Text HLabel 6400 1950 0    50   Input ~ 0
 ~RAMRD
 Wire Wire Line
-	8300 1600 8200 1600
-Wire Wire Line
-	7600 1500 7500 1500
-Wire Wire Line
-	7500 1500 7500 1350
-Wire Wire Line
-	7500 1350 7400 1350
-Wire Wire Line
-	7400 1850 7500 1850
-Wire Wire Line
-	7500 1850 7500 1700
-Wire Wire Line
-	7500 1700 7600 1700
-Wire Wire Line
-	6800 1250 6700 1250
-Wire Wire Line
-	6100 1250 6000 1250
-Wire Wire Line
-	6000 1950 6800 1950
-Wire Wire Line
-	6700 1600 6700 1450
-Wire Wire Line
-	6700 1450 6800 1450
-Connection ~ 6700 1600
-Wire Wire Line
-	6700 1600 6000 1600
-Text Notes 6500 800  0    50   ~ 0
-Allow RAM output during video cycles via ~CAS~.\nDuring CPU cycles guard against clashes with ~MWE~.
-Wire Wire Line
-	6700 1600 6700 1750
-Wire Wire Line
-	6700 1750 6800 1750
+	8000 1600 7900 1600
+Wire Wire Line
+	7300 1500 7200 1500
+Wire Wire Line
+	7200 1500 7200 1350
+Wire Wire Line
+	7100 1850 7200 1850
+Wire Wire Line
+	7200 1850 7200 1700
+Wire Wire Line
+	7200 1700 7300 1700
+Wire Wire Line
+	6400 1950 6500 1950
+Text Notes 6100 1200 0    50   ~ 0
+Ensure ~RAMOE~ doesn't clash with ~RAMWE~.\nDuring CPU cycles, only allow RAM to output (~RAMOE~) when\n~RAMRD~ is active. During video cycles hold ~RAMOE~ active.\nRAM reads will be enabled or disabled by ~RAMCS~.\nThis could be improved but it works.
 $Comp
 L 74xx:74LS08 U193
@@
 Text Notes 4200 1900 0    100  ~ 0
 RAM CONTROL
-Text Notes 4300 3200 0    100  ~ 0
-EXP RAM CONTROL
+Text Notes 2850 2850 0    100  ~ 0
+EXPANSION RAM CONTROL
 Text HLabel 8800 1750 1    50   3State ~ 0
 DATA_BUS
@@
 $Comp
 L 74xx:74LS04 U191
-U 6 1 638768EC
-P 6400 1250
-F 0 "U191" H 6400 1567 50  0000 C CNN
-F 1 "74LS04" H 6400 1476 50  0000 C CNN
-F 2 "Package_DIP:DIP-14_W7.62mm_Socket" H 6400 1250 50  0001 C CNN
-F 3 "http://www.ti.com/lit/gpn/sn74LS04" H 6400 1250 50  0001 C CNN
-	6    6400 1250
-	1    0    0    -1
-$EndComp
-$Comp
-L 74xx:74LS04 U191
 U 7 1 63876F1A
 P 6450 4750
@@
 L power:GND #PWR?
 U 1 1 63899CAD
-P 6150 7500
+P 6150 7650
 AR Path="/63899CAD" Ref="#PWR?"  Part="1"
 AR Path="/6071ED56/63899CAD" Ref="#PWR?"  Part="1"
 AR Path="/60F2930F/63899CAD" Ref="#PWR0123"  Part="1"
-F 0 "#PWR0123" H 6150 7250 50  0001 C CNN
-F 1 "GND" H 6000 7450 50  0001 C CNN
-F 2 "" H 6150 7500 50  0001 C CNN
-F 3 "" H 6150 7500 50  0001 C CNN
-	1    6150 7500
+F 0 "#PWR0123" H 6150 7400 50  0001 C CNN
+F 1 "GND" H 6000 7600 50  0001 C CNN
+F 2 "" H 6150 7650 50  0001 C CNN
+F 3 "" H 6150 7650 50  0001 C CNN
+	1    6150 7650
 	1    0    0    -1
 $EndComp
@@
 NoConn ~ 6750 6900
 Wire Wire Line
-	6150 6150 6150 6800
-Wire Wire Line
-	6150 7000 6150 7500
-Text HLabel 2400 2150 0    50   Input ~ 0
+	6150 6150 6150 6450
+Wire Wire Line
+	6150 7000 6150 7300
+Text HLabel 2550 2250 0    50   Input ~ 0
 ~CPU_ADDR
 Wire Wire Line
-	3300 2150 3200 2150
-Wire Wire Line
-	2400 2150 2500 2150
-Wire Wire Line
-	2500 2150 2500 2050
-Wire Wire Line
-	2500 2050 2600 2050
-Wire Wire Line
-	2500 2150 2500 2250
-Wire Wire Line
-	2500 2250 2600 2250
-Connection ~ 2500 2150
+	2550 2250 2650 2250
+Wire Wire Line
+	2650 2250 2650 2150
+Wire Wire Line
+	2650 2150 2750 2150
+Wire Wire Line
+	2650 2250 2650 2350
+Wire Wire Line
+	2650 2350 2750 2350
+Connection ~ 2650 2250
+Wire Wire Line
+	2450 1400 2800 1400
+Text Label 2800 1400 2    50   ~ 0
+XCPU_AD
+Text Label 6850 1350 0    50   ~ 0
+XCPU_AD
+Text Label 6100 1750 0    50   ~ 0
+~XCPU_AD
+Wire Wire Line
+	6100 1750 6500 1750
+Wire Wire Line
+	6850 1350 7200 1350
+Text Notes 2550 1850 0    50   ~ 0
+Buffer ~CPU_ADDR~ for signal\nintegrity reasons
+Text Label 3900 2250 2    50   ~ 0
+~BUF_CPU_AD
+Text Label 1200 900  0    50   ~ 0
+~BUF_CPU_AD
+Text Label 3150 1100 0    50   ~ 0
+~BUF_CPU_AD
+Wire Wire Line
+	3150 1100 3700 1100
+Wire Wire Line
+	1700 900  1200 900
+Wire Wire Line
+	3350 2250 3900 2250
+Text Label 1700 4300 0    50   ~ 0
+~BUF_CPU_AD
+Wire Wire Line
+	1700 4300 2250 4300
+$Comp
+L 74xx:74LS32 U192
+U 4 1 651FD105
+P 6450 7400
+F 0 "U192" H 6450 7725 50  0000 C CNN
+F 1 "74LS32" H 6450 7634 50  0000 C CNN
+F 2 "Package_DIP:DIP-14_W7.62mm_Socket" H 6450 7400 50  0001 C CNN
+F 3 "http://www.ti.com/lit/gpn/sn74LS32" H 6450 7400 50  0001 C CNN
+	4    6450 7400
+	1    0    0    -1
+$EndComp
+Wire Wire Line
+	6150 7650 6150 7500
+Connection ~ 6150 7300
+Connection ~ 6150 7500
+Wire Wire Line
+	6150 7500 6150 7300
+$Comp
+L 74xx:74LS04 U191
+U 6 1 6520CC2A
+P 6450 6450
+F 0 "U191" H 6450 6767 50  0000 C CNN
+F 1 "74LS04" H 6450 6676 50  0000 C CNN
+F 2 "Package_DIP:DIP-14_W7.62mm_Socket" H 6450 6450 50  0001 C CNN
+F 3 "http://www.ti.com/lit/gpn/sn74LS04" H 6450 6450 50  0001 C CNN
+	6    6450 6450
+	1    0    0    -1
+$EndComp
+Connection ~ 6150 6450
+Wire Wire Line
+	6150 6450 6150 6800
+NoConn ~ 6750 6450
+NoConn ~ 6750 7400
 Wire Bus Line
 	1100 2900 1500 2900
@@
 Wire Bus Line
 	8800 1750 8800 4600
-Text GLabel 3600 1100 0    50   Input ~ 0
-~CPU_ADDRx
-Text GLabel 950  900  0    50   Input ~ 0
-~CPU_ADDRx
-Text GLabel 3300 2150 2    50   Output ~ 0
-~CPU_ADDRx
-Text GLabel 2250 4300 0    50   Input ~ 0
-~CPU_ADDRx
 $EndSCHEMATC

Commit message: Long overdue update...
Parts:
- renumbered U192 to IC192
Connections:
- net D0: now also U114.12 (O4), U115.8 (I3a); no longer U114.19 (O7), U115.2 (I0a)
- net D1: now also U114.9 (O3), U115.11 (I0b); no longer U114.2 (O0), U115.17 (I3b)
- net D2: now also U114.15 (O5), U115.6 (I2a); no longer U114.16 (O6), U115.4 (I1a)
- net D3: now also U114.6 (O2), U115.13 (I1b), U194.12 (D2); no longer U114.5 (O1), U115.15 (I2b), U194.14 (D0)
- net D4: now also U114.16 (O6), U115.4 (I1a); no longer U114.15 (O5), U115.6 (I2a)
- net D5: now also U114.5 (O1), U115.15 (I2b), U194.14 (D0); no longer U114.6 (O2), U115.13 (I1b), U194.12 (D2)
- net D6: now also U114.19 (O7), U115.2 (I0a); no longer U114.12 (O4), U115.8 (I3a), U194.11 (D3)
- net D7: now also U114.2 (O0), U115.17 (I3b); no longer U114.9 (O3), U115.11 (I0b)
- net GND: now also IC192.1, IC192.2, U194.11 (D3); no longer IC112.1, IC112.2
- net RAMA16: now also R194.2, U194.5 (Q2); no longer R192.2, U194.3 (Q0)
- net RAMA18: now also R192.2, U194.3 (Q0); no longer R194.2, U194.5 (Q2)
- net ~IORQ: now also IC112.1; no longer IC112.12
- net ~RAMRD: now also IC112.12; no longer IC192.2
- net ~WR: now also IC112.2; no longer IC112.13
- net ~XCPU_AD: now also IC112.13; no longer IC192.1
- net at IC118.18 (~IOWR), U194.7 (Cp): now also IC112.3; no longer IC112.11
- net at U193.2: now also IC112.11; no longer IC192.3
- net RAMA14 renamed AOUT14
- net RAMA15 renamed AOUT15
- net RAMD0 renamed RD6
- net RAMD1 renamed RD7
- net RAMD2 renamed RD4
- net RAMD3 renamed RD5
- net RAMD4 renamed RD2
- net RAMD5 renamed RD3
- net RAMD6 renamed RD0
- net RAMD7 renamed RD1
Other:
- moved on the sheet: IC112A, IC112D, IC192A
