File: ROM/CPCROM.sch (KiCad schematic (older format))
At the start: 13 parts, among them IC191 74LS32, IC192 74LS32, IC193 74LS02, IC194 74LS08, IC195 74LS74

Commit message: Long overdue update...
Parts:
- removed C6: 0.1nF, Capacitor_THT:C_Disc_D3.0mm_W2.0mm_P2.50mm, symbol Device:C
- removed unit 3 of IC193
- removed unit 4 of IC193
- removed unit 2 of IC193
- removed unit 2 of IC194
- removed unit 2 of IC195
- removed JP1: RC2014Bus, Connector_PinHeader_2.54mm:PinHeader_1x40_P2.54mm_Vertical, symbol CPCROM-rescue:RC2014Bus-CPC
- added JP1: Conn_02x25_Odd_Even, Connector_IDC:IDC-Header_2x25_P2.54mm_Horizontal, symbol Connector_Generic:Conn_02x25_Odd_Even
Connections:
- net +5V: now also JP1.24 (Pin_24)
- net A0: now also JP1.33 (Pin_33)
- net A1: now also JP1.34 (Pin_34)
- net A10: now also JP1.43 (Pin_43)
- net A11: now also JP1.44 (Pin_44)
- net A12: now also JP1.45 (Pin_45)
- net A13: now also JP1.46 (Pin_46)
- net A15: now also JP1.48 (Pin_48)
- net A2: now also JP1.35 (Pin_35)
- net A3: now also JP1.36 (Pin_36)
- net A4: now also JP1.37 (Pin_37)
- net A5: now also JP1.38 (Pin_38)
- net A6: now also JP1.39 (Pin_39)
- net A7: now also JP1.40 (Pin_40)
- net A8: now also JP1.41 (Pin_41)
- net A9: now also JP1.42 (Pin_42)
- net D0: now also JP1.25 (Pin_25)
- net D1: now also JP1.26 (Pin_26)
- net D2: now also JP1.27 (Pin_27)
- net D3: now also JP1.28 (Pin_28)
- net D4: now also JP1.29 (Pin_29)
- net D5: now also JP1.30 (Pin_30)
- net D6: now also JP1.31 (Pin_31)
- net D7: now also JP1.32 (Pin_32)
- net GND: now also JP1.2 (Pin_2), JP1.49 (Pin_49)
- net ROMDIS: now also JP1.8 (Pin_8)
- net ~ROMEN: now also JP1.9 (Pin_9)
- new net RAMDIS: JP1.6 (Pin_6)
- new net ~IORQ: JP1.20 (Pin_20)
- new net ~MREQ: JP1.23 (Pin_23)
- new net ~RD: JP1.19 (Pin_19)
- new net ~RESET: JP1.10 (Pin_10)
- new net ~WR: JP1.18 (Pin_18)
- no-connect marks 14 -> 16
