File: ROM/ROM.sch (KiCad schematic (older format))
At the start: 18 parts, among them IC103 SST39SF040, IC190 74LS374, IC191 74LS32, IC192 74LS32, IC193 74LS02, IC194 74LS08, IC195 74LS74

Commit message: Long overdue update...
Parts:
- removed LK2, LK3, LK4, LK5: Jumper_NO_Small, Connector_PinHeader_2.54mm:PinHeader_1x02_P2.54mm_Vertical, symbol Device:Jumper_NO_Small
- added D190: ARMED, LED_THT:LED_D3.0mm, symbol Device:LED
- added D191: ENABLED, LED_THT:LED_D3.0mm, symbol Device:LED
- added D192: WRITE, LED_THT:LED_D3.0mm, symbol Device:LED
- added D193: 1N4148, Diode_THT:D_DO-35_SOD27_P7.62mm_Horizontal, symbol Diode:1N4148
- added unit 1 of IC193
- added unit 4 of IC193
- added unit 2 of IC193
- added unit 2 of IC194
- added unit 2 of IC195
- added JP2, JP3, JP4, JP5, JP6, JP7: Jumper_NC_Small, Jumper:SolderJumper-2_P1.3mm_Bridged_RoundedPad1.0x1.5mm, symbol Device:Jumper_NC_Small
- added R195, R196, R197: 2k2, Resistor_THT:R_Axial_DIN0207_L6.3mm_D2.5mm_P7.62mm_Horizontal, symbol Device:R
- added R198, R199, R200: 470, Resistor_THT:R_Axial_DIN0207_L6.3mm_D2.5mm_P7.62mm_Horizontal, symbol Device:R
- LK1: value Jumper_NO_Small -> RAMDIS
Connections:
- net +5V: now also D190.2 (A), D192.2 (A), IC195.10 (~S)
- net A15: now also IC193.8; no longer IC193.2
- net D7: now also IC195.2 (D)
- net GND: now also JP2.2, JP3.2, JP4.2, JP5.2, JP6.2, JP7.2, R195.1, R196.1, R197.1, R199.2
- net ROMDIS: now also IC192.5, R112.1
- net WRITE_EN: now also D191.2 (A), IC195.9 (Q); no longer IC192.2, IC193.3, IC195.5 (Q)
- net ~IORQ: now also IC192.1; no longer IC191.5
- net ~MREQ: now also IC192.13; no longer IC192.10
- net ~RD: now also IC103.24 (OE); no longer IC192.1
- net ~ROMEN: now also IC192.4; no longer IC192.5
- net ~WR: now also IC192.10, IC192.2; no longer IC191.4, IC192.13
- net ~WRITE_EN: now also IC192.9, IC195.8 (~Q); no longer IC192.12, IC195.6 (~Q)
- net at IC103.22 (CE), IC194.3: no longer LK1.2
- net at IC192.3: now also IC191.10; no longer IC103.24 (OE)
- net ~WRITE: now reaches IC103.31 (PGM), IC194.1
- net ~WRITE: now also IC192.11, IC193.5, IC193.6, IC194.4, IC194.5; no longer IC192.8
- net at IC190.1 (OE): now also IC193.10; no longer IC193.1
- net at IC190.15 (O5): now also IC194.13, R197.2; no longer IC194.12
- net at IC190.16 (O6): now also IC194.12, R196.2; no longer IC194.13
- net at IC190.19 (O7), IC194.10: now also R195.2
- net at IC191.6: no longer IC191.10
- net at IC194.8: now also IC195.12 (D); no longer IC195.2 (D)
- net at IC191.11, IC195.3 (C): now also IC195.11 (C)
- net at IC192.6, IC194.2: no longer LK1.1
- new net: IC191.4, JP6.1
- new net: IC191.5, JP7.1
- new net: IC192.12, IC192.8
- new net: D193.1 (K), LK1.1
- new net: IC193.2, JP4.1
- new net: IC193.3, JP5.1
- new net: IC193.11, JP2.1
- new net: IC193.12, JP3.1
- new net: D193.2 (A), IC193.4
- new net: D190.1 (K), R198.1
- new net: D191.1 (K), R199.1
- new net: D192.1 (K), R200.1
- new net: IC194.6, R200.2
- new net ARMED: IC193.9, IC195.13 (~R), IC195.5 (Q)
- new net RAMDIS: LK1.2
- new net ~ARMED: IC195.6 (~Q), R198.2
- no-connect marks 0 -> 3
Other:
- note added: "HOW TO FLASH THE EEPROM\n\nout (&cfff),ROM_number OR $e0 ;Arm\n<repeat above instruction> ;Write enable\n<Program FLASH as per datasheet>\nout (&cfff),ROM_number ;Disable and disarm\n\nWhen write enabled:\n* A15 and A14 are ignored.\n* The flash maps to *all* memory banks.\n* Writes to RAM are disbled (if LK1 installed).\n* Firmware is in bank 31.\n\nROM burning code *must* run from RAM.\nInterru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"
- note added: "Memory writes when ~WRITE_EN~ is active \nwill write to ROM."
- note added: "ROM slot 31 is firmware\nSlots 0..30 are upper ROMs\n\nPorts:\nROM select: &dfff\nWrite control: &cfff"
- note added: "THIS NO LONGER APPLIES\n\n!!!\nThere is no way to disable memory writes on the standard CPC system. Therefore ANY \nmemory writes which we do to ROM while WRITE_EN is active will also write to RAM.\n\nHowever, since the ROM maps to any and all memory banks this adds a certain \namount of flexibility. Also note that reading from ROM is disabled whilst writing is \nenabled. This means we can read f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"
- note added: "We also want to enable the outputs \nwhen 'armed'."
- note added: "When ARMED IC190 will be permanently enabled\n(and outputting selected address)"
- note removed: "!!!\nThere is no way to disable memory writes on the standard CPC system. Therefore ANY \nmemory writes which we do to ROM while WRITE_EN is active will also write to RAM.\n\nHowever, since the ROM maps to any and all memory banks this adds a certain \namount of flexibility. Also note that reading from ROM is disabled whilst writing is \nenabled. This means we can read from the RAM 'underneath' t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"
- note removed: "For CPC: install links LK4 and LK5 (permanently \ndisables/overrides onboard ROM).\nFor CPC modular: Install link from LK4 to LK5."
- note removed: "Latch on port &efff"
- note removed: "Memory writes when ~WRITE_EN~ is active \nwill write to ROM (and RAM!!)"
- note removed: "To disable write feature (or save cost), leave out IC194 and IC195 \nand install jumpers on links LK1, LK2 and LK3."
- note removed: "WRITE_EN will inhibit reads while enabled.\n(Not strictly necessary)."
- note removed: "We also want to enable the outputs \nwhen write enabling is active."
- moved on the sheet: IC191B, IC191D, IC192A, IC192B, IC194A, IC194C, IC194D, IC195A, LK1, R112
