File: Sound/CPCSound.kicad_pcb (KiCad board)
At the start: 2 copper layers, 99.1 x 52.9 mm, 28 parts, among them IC101 74LS145, IC102 AY-3-8910, J102 Paddle Port (9-Pin D), J103 AudioJack3_Ground_SwitchTR, J192 Paddle Port 2 (9-Pin D), J193 Conn_01x09_Male, J903 Conn_01x08_Female, X1 CXO_DIP14_1MHz

Commit message: Long overdue update...
Parts:
- removed CP2: Keyboard Connector (20-way inline 2.54mm), Connector_PinHeader_2.54mm:PinHeader_1x20_P2.54mm_Vertical
- removed J903: Conn_01x08_Female, Connector_PinSocket_2.54mm:PinSocket_1x08_P2.54mm_Vertical
- removed JP4: MIX, Connector_PinHeader_2.54mm:PinHeader_1x03_P2.54mm_Vertical
- removed JP5: LEFT, Connector_PinHeader_2.54mm:PinHeader_1x03_P2.54mm_Vertical
- removed JP6: RIGHT, Connector_PinHeader_2.54mm:PinHeader_1x03_P2.54mm_Vertical
- removed X1: CXO_DIP14_1MHz, Oscillator:Oscillator_DIP-14
- added D191: PESD5V0V1BA, Diode_SMD:D_SOD-323_HandSoldering, F.Cu at (210.2, 118.8)
- added D192: PESD5V0V1BA, Diode_SMD:D_SOD-323_HandSoldering, F.Cu at (212.7, 118.8)
- added D193: PESD5V0V1BA, Diode_SMD:D_SOD-323_HandSoldering, F.Cu at (215.3, 118.8)
- added D194: PESD5V0V1BA, Diode_SMD:D_SOD-323_HandSoldering, F.Cu at (217.8, 118.8)
- added D195: PESD5V0V1BA, Diode_SMD:D_SOD-323_HandSoldering, F.Cu at (220.3, 118.8)
- added D196: PESD5V0V1BA, Diode_SMD:D_SOD-323_HandSoldering, F.Cu at (222.9, 118.8)
- added D197: PESD5V0V1BA, Diode_SMD:D_SOD-323_HandSoldering, F.Cu at (226.7, 125.1)
- added D198: PESD5V0V1BA, Diode_SMD:D_SOD-323_HandSoldering, F.Cu at (226.7, 118.7)
- added D199: PESD5V0V1BA, Diode_SMD:D_SOD-323_HandSoldering, F.Cu at (229.2, 118.7)
- added D200: PESD5V0V1BA, Diode_SMD:D_SOD-323_HandSoldering, F.Cu at (231.8, 118.7)
- added D201: PESD5V0V1BA, Diode_SMD:D_SOD-323_HandSoldering, F.Cu at (231.8, 125.1)
- added D202: PESD5V0V1BA, Diode_SMD:D_SOD-323_HandSoldering, F.Cu at (229.2, 125.1)
- added D203: PESD5V0V1BA, Diode_SMD:D_SOD-323_HandSoldering, F.Cu at (224.2, 125.1)
- added D204: PESD5V0V1BA, Diode_SMD:D_SOD-323_HandSoldering, F.Cu at (221.6, 125.1)
- added D205: PESD5V0V1BA, Diode_SMD:D_SOD-323_HandSoldering, F.Cu at (219.1, 125.1)
- added D206: PESD5V0V1BA, Diode_SMD:D_SOD-323_HandSoldering, F.Cu at (216.5, 125.1)
- added D207: PESD5V0V1BA, Diode_SMD:D_SOD-323_HandSoldering, F.Cu at (214.0, 125.1)
- added D208: PESD5V0V1BA, Diode_SMD:D_SOD-323_HandSoldering, F.Cu at (211.5, 125.1)
- added D209: PESD5V0V1BA, Diode_SMD:D_SOD-323_HandSoldering, F.Cu at (169.5, 149.2)
- added D210: PESD5V0V1BA, Diode_SMD:D_SOD-323_HandSoldering, F.Cu at (169.6, 146.7)
- added D211: PESD5V0V1BA, Diode_SMD:D_SOD-323_HandSoldering, F.Cu at (169.5, 144.1)
- added D212: PESD5V0V1BA, Diode_SMD:D_SOD-323_HandSoldering, F.Cu at (169.6, 141.6)
- added D213: PESD5V0V1BA, Diode_SMD:D_SOD-323_HandSoldering, F.Cu at (169.6, 139.1)
- added D214: PESD5V0V1BA, Diode_SMD:D_SOD-323_HandSoldering, F.Cu at (169.5, 136.5)
- added D215: PESD5V0V1BA, Diode_SMD:D_SOD-323_HandSoldering, F.Cu at (169.5, 134.0)
- added D216: PESD5V0V1BA, Diode_SMD:D_SOD-323_HandSoldering, F.Cu at (169.5, 131.4)
- added D217: PESD5V0V1BA, Diode_SMD:D_SOD-323_HandSoldering, F.Cu at (169.5, 128.9)
- added D218: PESD5V0V1BA, Diode_SMD:D_SOD-323_HandSoldering, F.Cu at (163.8, 106.7)
- added D219: PESD5V0V1BA, Diode_SMD:D_SOD-323_HandSoldering, F.Cu at (166.4, 106.7)
- added D220: PESD5V0V1BA, Diode_SMD:D_SOD-323_HandSoldering, F.Cu at (237.5, 125.7)
- added D221: PESD5V0V1BA, Diode_SMD:D_SOD-323_HandSoldering, F.Cu at (237.5, 123.2)
- added D222: PESD5V0V1BA, Diode_SMD:D_SOD-323_HandSoldering, F.Cu at (243.8, 120.7)
- added D223: PESD5V0V1BA, Diode_SMD:D_SOD-323_HandSoldering, F.Cu at (237.5, 120.7)
- added D224: PESD5V0V1BA, Diode_SMD:D_SOD-323_HandSoldering, F.Cu at (243.8, 118.1)
- added D225: PESD5V0V1BA, Diode_SMD:D_SOD-323_HandSoldering, F.Cu at (237.5, 118.1)
- added D226: PESD5V0V1BA, Diode_SMD:D_SOD-323_HandSoldering, F.Cu at (243.8, 115.6)
- added D227: PESD5V0V1BA, Diode_SMD:D_SOD-323_HandSoldering, F.Cu at (237.5, 115.6)
- added RN901: 2k2, Resistor_THT:R_Array_SIP9, F.Cu at (231.8, 132.1)
- J103: value AudioJack3_Ground_SwitchTR -> AudioJack3_SwitchTR
- J192: footprint Connector_Dsub:DSUB-9_Male_Horizontal_P2.77x2.84mm_EdgePinOffset9.40mm -> Connector_Dsub:DSUB-9_Male_Horizontal_P2.77x2.84mm_EdgePinOffset9.90mm_Housed_MountingHolesOffset11.32mm
- J193: value Conn_01x09_Male -> Conn_01x10_Male; footprint Connector_PinHeader_2.54mm:PinHeader_1x09_P2.54mm_Vertical -> Connector_PinHeader_2.54mm:PinHeader_2x05_P2.54mm_Vertical
- JP1: value RC2014Bus -> CPCM_IOSound_EdgeBottom; footprint Connector_PinHeader_2.54mm:PinHeader_1x40_P2.54mm_Vertical -> CPCModular:Edge25_2.54PS; moved to B.Cu
- JP2: value RC2014ExtendedBus -> CPCM_IOSound_EdgeTop; footprint Connector_PinHeader_2.54mm:PinHeader_1x25_P2.54mm_Vertical -> CPCModular:Edge25_2.54PS
- JP3: value Osc sel -> Conn_02x10_Odd_Even; footprint Connector_PinHeader_2.54mm:PinHeader_1x03_P2.54mm_Vertical -> Connector_IDC:IDC-Header_2x10_P2.54mm_Vertical
- NT1: moved to F.Cu
- moved J102 77.5 mm to (162.6, 134.0), turned to 270 degrees
- moved J192 63.3 mm to (243.8, 144.8), turned to 90 degrees
- moved NT1 40.7 mm to (186.4, 107.3)
- moved J193 39.9 mm to (248.3, 109.9), turned to 0 degrees
- moved R121 39.0 mm to (177.2, 107.3), turned to 270 degrees
- moved R122 39.0 mm to (180.3, 107.3), turned to 270 degrees
- moved R123 39.0 mm to (183.5, 107.3), turned to 270 degrees
- moved IC102 38.3 mm to (189.9, 106.7), turned to 0 degrees
- moved JP3 35.3 mm to (237.5, 107.3), turned to 270 degrees
- moved JP2 30.2 mm to (172.7, 168.2)
- moved C1 29.3 mm to (208.3, 144.8), turned to 270 degrees
- moved R117 26.4 mm to (170.8, 114.9), turned to 90 degrees
- moved C2 26.0 mm to (213.4, 139.1)
- moved IC101 26.0 mm to (216.5, 146.7)
- moved R119 24.2 mm to (174.0, 117.5)
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Connections:
- net Net-(IC102-Pad9) renamed /IO_SOUND/AYB4
- net Net-(J103-PadR) renamed /IO_SOUND/SRIGHT
- net Net-(J103-PadT) renamed /IO_SOUND/SLEFT
- IC102 pad 10: Net-(IC102-Pad10) -> /IO_SOUND/AYB3
- IC102 pad 11: Net-(IC102-Pad11) -> /IO_SOUND/AYB2
- IC102 pad 12: Net-(IC102-Pad12) -> /IO_SOUND/AYB1
- IC102 pad 13: Net-(IC102-Pad13) -> /IO_SOUND/AYB0
- IC102 pad 22: Net-(IC102-Pad22) -> /IO_SOUND/SOUND_CLK
- IC102 pad 6: Net-(IC102-Pad6) -> /IO_SOUND/AYB7
- IC102 pad 7: Net-(IC102-Pad7) -> /IO_SOUND/AYB6
- IC102 pad 8: Net-(IC102-Pad8) -> /IO_SOUND/AYB5
- J192 pad 9: /IO_SOUND/COMMON -> Net-(J192-Pad9)
- J193 pad 2: Net-(IC102-Pad13) -> GND
- J193 pad 3: Net-(IC102-Pad12) -> /IO_SOUND/AYB7
- J193 pad 4: Net-(IC102-Pad11) -> /IO_SOUND/AYB6
- J193 pad 5: Net-(IC102-Pad10) -> /IO_SOUND/AYB5
- J193 pad 7: Net-(IC102-Pad8) -> /IO_SOUND/AYB3
- J193 pad 8: Net-(IC102-Pad7) -> /IO_SOUND/AYB2
- J193 pad 9: Net-(IC102-Pad6) -> /IO_SOUND/AYB1
- JP1 pad 1: Net-(JP1-Pad1) -> GND
- JP1 pad 10: Net-(JP1-Pad10) -> PA2
- JP1 pad 11: Net-(JP1-Pad11) -> PA4
- JP1 pad 12: Net-(JP1-Pad12) -> PA6
- JP1 pad 17: GND -> Net-(JP1-Pad17)
- JP1 pad 18: +5V -> /IO_SOUND/BDIR
- JP1 pad 19: Net-(JP1-Pad19) -> /IO_SOUND/BC1
- JP1 pad 20: /IO_SOUND/~RESET -> Net-(JP1-Pad20)
- JP1 pad 21: Net-(JP1-Pad21) -> PC0
- JP1 pad 22: Net-(JP1-Pad22) -> PC2
- JP1 pad 23: Net-(JP1-Pad23) -> /IO_SOUND/SOUND_CLK
- JP1 pad 3: Net-(JP1-Pad3) -> /IO_SOUND/ARIGHT
- JP1 pad 9: Net-(JP1-Pad9) -> PA0
- JP2 pad 1: GND -> /IO_SOUND/SOUND
- JP2 pad 10: Net-(JP2-Pad10) -> PA3
- JP2 pad 11: PA0 -> PA5
- JP2 pad 12: PA1 -> PA7
- JP2 pad 13: PA2 -> Net-(JP2-Pad13)
- JP2 pad 14: PA3 -> Net-(JP2-Pad14)
- JP2 pad 15: PA4 -> Net-(JP2-Pad15)
- JP2 pad 16: PA5 -> Net-(JP2-Pad16)
- JP2 pad 17: PA6 -> +5V
- JP2 pad 18: PA7 -> Net-(JP2-Pad18)
- JP2 pad 2: +5V -> Net-(JP2-Pad2)
- JP2 pad 21: Net-(JP2-Pad21) -> /IO_SOUND/~RESET
- JP2 pad 22: Net-(JP2-Pad22) -> PC1
- JP2 pad 23: Net-(JP2-Pad23) -> PC3
- JP2 pad 25: (no net) -> GND
- JP2 pad 3: Net-(JP2-Pad3) -> /IO_SOUND/ALEFT
- JP2 pad 5: /IO_SOUND/SOUND_CLK -> Net-(JP2-Pad5)
- JP2 pad 9: Net-(JP2-Pad9) -> PA1
- JP3 pad 1: Net-(JP3-Pad1) -> /IO_SOUND/COMMON
- JP3 pad 2: Net-(IC102-Pad22) -> Net-(JP3-Pad2)
- JP3 pad 3: /IO_SOUND/SOUND_CLK -> /IO_SOUND/Y9
Routing:
- net GND: track 28.6 -> 535.4 mm, vias 0 -> 23
- net /IO_SOUND/COM_2: track 33.1 -> 168.2 mm, vias 0 -> 2
- net /IO_SOUND/AYA0: track 47.2 -> 162.5 mm, vias 1 -> 3
- net +5V: track 2.54 -> 105.0 mm, vias 0 -> 1
- net /IO_SOUND/COMMON: track 36.2 -> 137.1 mm
- net Net-(JP2-Pad20): track 97.8 -> 0.00 mm
- net Net-(JP1-Pad36): track 97.1 -> 0.00 mm
- net Net-(JP2-Pad19): track 95.9 -> 0.00 mm, vias 1 -> 0
- net Net-(JP1-Pad35): track 94.6 -> 0.00 mm
- net /IO_SOUND/AYA1: track 57.2 -> 148.3 mm, vias 1 -> 3
- net /IO_SOUND/AYB0: track 0.00 -> 74.7 mm, vias 0 -> 1
- net /IO_SOUND/AYA5: track 59.1 -> 133.7 mm, vias 0 -> 2
- net /IO_SOUND/AYA2: track 59.3 -> 133.3 mm, vias 1 -> 2
- net /IO_SOUND/AYA6: track 52.6 -> 124.0 mm, vias 0 -> 2
- net /IO_SOUND/AYA4: track 57.2 -> 127.9 mm, vias 0 -> 3
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- added copper zone on F.Cu, net GND
- added copper zone on F.Cu, net GNDA
- removed copper zone on F.Cu, net +5V
- removed copper zone on B.Cu, net GNDA
Other:
- board size 99.1 x 52.9 mm -> 99.1 x 71.1 mm
- board text added: "All SMT diodes are PESD5V0V1BA. These are bidirectional, so ignore polarity when installing. They are for ESD protection and recommended but the board will work without them. All capacitors are 100nF unless marked."
- board text added: "CPC Modular Sound module © Mike Sutton 2024 Bread80.com @bread80@mstdn.social"
- board text added: "D191..D208"
- board text added: "D209..D217"
- board text added: "D220..D227"
- board text added: "JOYSTICK 2"
- board text added: "Keyboard connector pinout matches that of the CPC6128. 'Left' and 'Right' refer to connector positioning on the '6128 motherboard."
- board text added: "Only if required"
- board text added: "REV 2"
- board text added: "RN901: If using AY-3-8910: Do not install AY-3-8910A: Install"
- board text added: "by Bread80"
- board text removed: "--- AY BUS 0..7 ---"
- board text removed: "A15 A14 A13 A12 A11 A10 A9 A8 A7 A6 A5 A4 A3 A2 A1 A0 Gnd 5v M1 Reset Clock INT Mreq Wr Ro IORQ D0 D1 D2 D3 D4 D5 D6 D7 Tx Rx USR1 USR2 USR3"
- board text removed: "BACKPLANE OUT SELECT"
- board text removed: "Bread80.com"
- board text removed: "CLK2"
- board text removed: "CLOCK SELECT"
- board text removed: "CPC Modular for RC2014 backplane Sound module © Mike Sutton 2022 Bread80.com @bread80@mstdn.social"
- board text removed: "MIX"
- board text removed: "OSC"
- board text removed: "Pin 1"
- board text removed: "REV 0.1"
- board text removed: "RX"
- board text removed: "RX2"
- board text removed: "Rx2/Rx"
- board text removed: "TX"
- board text removed: "TX2"
- board text removed: "Tx2/Tx"
