File: Sound/IO_SOUND.sch (KiCad schematic (older format))
At the start: 20 parts, among them IC101 74LS145, IC102 AY-3-8910, J102 Paddle Port (9-Pin D), J103 AudioJack3_Ground_SwitchTR, J192 Paddle Port 2 (9-Pin D), J193 Conn_01x09_Male, X1 CXO_DIP14_1MHz

Commit message: Long overdue update...
Parts:
- removed CP002: Keyboard Connector (20-way inline 2.54mm), Connector_PinHeader_2.54mm:PinHeader_1x20_P2.54mm_Vertical, symbol Connector:Conn_01x20_Male
- removed J103: AudioJack3_Ground_SwitchTR, Connector_Audio:Jack_3.5mm_CUI_SJ1-3535NG_Horizontal, symbol Connector:AudioJack3_Ground_SwitchTR
- removed JP3: Osc sel, Connector_PinHeader_2.54mm:PinHeader_1x03_P2.54mm_Vertical, symbol Jumper:Jumper_3_Bridged12
- removed X1: CXO_DIP14_1MHz, Oscillator:Oscillator_DIP-14, symbol Oscillator:CXO_DIP14
- added D191, D192, D193, D194, D195, D196, D197, D198, D199, D200, D201, D202, D203, D204, D205, D206, D207, D208, D209, D210, D211, D212, D213, D214, D215, D216, D217, D218, D219, D220, D221, D222, D223, D224, D225, D226, D227: PESD5V0V1BA, Diode_SMD:D_SOD-323_HandSoldering, symbol Device:D_TVS_ALT
- added J103: AudioJack3_SwitchTR, Connector_Audio:Jack_3.5mm_CUI_SJ1-3535NG_Horizontal, symbol Connector:AudioJack3_SwitchTR
- added JP3: Conn_02x10_Odd_Even, Connector_IDC:IDC-Header_2x10_P2.54mm_Vertical, symbol Connector_Generic:Conn_02x10_Odd_Even
- added RN901: 2k2, Resistor_THT:R_Array_SIP9, symbol Device:R_Network08
- J192: footprint Connector_Dsub:DSUB-9_Male_Horizontal_P2.77x2.84mm_EdgePinOffset9.40mm -> Connector_Dsub:DSUB-9_Male_Horizontal_P2.77x2.84mm_EdgePinOffset9.90mm_Housed_MountingHolesOffset11.32mm
- J193: value Conn_01x09_Male -> Conn_01x10_Male; footprint Connector_PinHeader_2.54mm:PinHeader_1x09_P2.54mm_Vertical -> Connector_PinHeader_2.54mm:PinHeader_2x05_P2.54mm_Vertical; symbol Connector:Conn_01x09_Male -> Connector:Conn_01x10_Male
Connections:
- net +5V: now also RN901.1 (common)
- net ALEFT: now also J103.TN
- net ARIGHT: now also J103.RN
- net AYA0: now also D201.1 (A1), D209.1 (A1), JP3.4 (Pin_4), RN901.2 (R1)
- net AYA1: now also D202.1 (A1), D210.1 (A1), JP3.6 (Pin_6), RN901.3 (R2)
- net AYA2: now also D203.1 (A1), D213.1 (A1), JP3.8 (Pin_8), RN901.4 (R3)
- net AYA3: now also D204.1 (A1), D212.1 (A1), JP3.10 (Pin_10), RN901.5 (R4)
- net AYA4: now also D205.1 (A1), D215.1 (A1), JP3.12 (Pin_12), RN901.6 (R5)
- net AYA5: now also D206.1 (A1), D214.1 (A1), JP3.14 (Pin_14), RN901.7 (R6)
- net AYA6: now also D207.1 (A1), D211.1 (A1), JP3.16 (Pin_16), RN901.8 (R7)
- net AYA7: now also D208.1 (A1), JP3.18 (Pin_18), RN901.9 (R8)
- net COMMON: now also D200.1 (A1), D217.1 (A1), JP3.1 (Pin_1); no longer J192.9
- net COM_2: now also D197.1 (A1), D216.1 (A1), JP3.7 (Pin_7)
- net GND: now also J193.2 (Pin_2), D191.2 (A2), D192.2 (A2), D193.2 (A2), D194.2 (A2), D195.2 (A2), D196.2 (A2), D197.2 (A2), D198.2 (A2), D199.2 (A2), D200.2 (A2), D201.2 (A2), D202.2 (A2), D203.2 (A2), D204.2 (A2), D205.2 (A2), D206.2 (A2), D207.2 (A2), D208.2 (A2), D209.2 (A2), D210.2 (A2), D211.2 (A2), D212.2 (A2), D213.2 (A2), D214.2 (A2), D215.2 (A2), D216.2 (A2), D217.2 (A2), D220.2 (A2), D221.2 (A2), D222.2 (A2), D223.2 (A2), D224.2 (A2), D225.2 (A2), D226.2 (A2), D227.2 (A2)
- net GNDA: now also D218.2 (A2), D219.2 (A2), J103.S
- net SOUND_CLK: now also IC102.22 (CLOCK)
- net Y1: now also D191.1 (A1), JP3.19 (Pin_19)
- net Y2: now also D192.1 (A1), JP3.17 (Pin_17)
- net Y3: now also D193.1 (A1), JP3.15 (Pin_15)
- net Y4: now also D194.1 (A1), JP3.13 (Pin_13)
- net Y5: now also D195.1 (A1), JP3.11 (Pin_11)
- net Y6: now also D196.1 (A1), JP3.9 (Pin_9)
- net Y8: now also D198.1 (A1), JP3.5 (Pin_5)
- net Y9: now also D199.1 (A1), JP3.3 (Pin_3)
- net SRIGHT: now reaches R117.1, R118.1
- net SRIGHT: now also D219.1 (A1), J103.R
- net SLEFT: now reaches R119.1, R120.1
- net SLEFT: now also D218.1 (A1), J103.T
- net AYB3: now reaches IC102.10 (IOB3)
- net AYB3: now also J193.7 (Pin_7), D223.1 (A1); no longer J193.5 (Pin_5)
- net AYB2: now reaches IC102.11 (IOB2)
- net AYB2: now also J193.8 (Pin_8), D222.1 (A1); no longer J193.4 (Pin_4)
- net AYB1: now reaches IC102.12 (IOB1)
- net AYB1: now also J193.9 (Pin_9), D221.1 (A1); no longer J193.3 (Pin_3)
- net AYB0: now reaches IC102.13 (IOB0)
- net AYB0: now also J193.10 (Pin_10), D220.1 (A1); no longer J193.2 (Pin_2)
- net AYB7: now reaches IC102.6 (IOB7)
- net AYB7: now also J193.3 (Pin_3), D227.1 (A1); no longer J193.9 (Pin_9)
- net AYB6: now reaches IC102.7 (IOB6)
- net AYB6: now also J193.4 (Pin_4), D226.1 (A1); no longer J193.8 (Pin_8)
- net AYB5: now reaches IC102.8 (IOB5)
- net AYB5: now also J193.5 (Pin_5), D225.1 (A1); no longer J193.7 (Pin_7)
- net AYB4: now reaches IC102.9 (IOB4), J193.6 (Pin_6)
- net AYB4: now also D224.1 (A1)
- no-connect marks 3 -> 5
Other:
- note added: "(Original CPC464 keyboard connector)"
- note added: "6128 left\nhand connector"
- note added: "6128 right\nhand connector"
- note added: "Modifications\n---\nReplaced the AY-3-8912 with a '8910 (because they're cheaper).\nThe extra port B has been brought out to header pins in case you \nwant to use it (see below).\nA second joystick port has been added.\nSound outputs to the bus as both separate left and right signals \nand stereo mix. This allows, for example, for an amplifier board \nand on board speaker. It should also be possi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"
- note added: "NOTE: Connector rows (left/right)\nare flipped on the PCB to make cabling \ncompatible with the CPC Modular keyboard."
- note added: "Optional pull-ups. Only for\nAY variants which don't have \nthem internally."
- note added: "TVS diodes (SMT)"
- note removed: "Modifications\n---\nReplaced the AY-3-8912 with a '8910 (because they're cheaper).\nThe extra port B has been brought out to header pins in case you want to use it (see \nbelow).\nThe parallel port has been deleted.\nA jumpers (LK5, LK6, LK7) has been added so the old parallel port busy signal \nand two of the (region) config lines can be reused to drive the '8910's extra \ncontrol lines.\nA seco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"
- note removed: "Stereo channels may be the \nwrong way round."
