File: Video/CPCVideo.kicad_pcb (KiCad board)
At the start: 2 copper layers, 99.1 x 52.9 mm, 29 parts, among them IC118 AMG40007, IC918 AMG40010, J1 VIDEO OUT, Q102 2SC1815Y, Q103 2N2369, X901 16MHz CXO_DIP14

Commit message: Long overdue update...
Parts:
- removed ?: , Mounting_Holes:MountingHole_3.2mm_M3
- removed JP901: Conn_01x10_Male, Connector_PinHeader_2.54mm:PinHeader_1x10_P2.54mm_Vertical
- added C139: 220p, Capacitor_THT:C_Disc_D3.0mm_W1.6mm_P2.50mm, F.Cu at (175.9, 134.0)
- added C140: 220p, Capacitor_THT:C_Disc_D3.0mm_W1.6mm_P2.50mm, F.Cu at (175.9, 124.5)
- added C141: 220p, Capacitor_THT:C_Disc_D3.0mm_W1.6mm_P2.50mm, F.Cu at (175.9, 114.9)
- added C901: 1uF, Capacitor_THT:CP_Radial_D7.5mm_P2.50mm, F.Cu at (185.4, 144.8)
- added D901: PESD5V0V1BA, Diode_SMD:D_SOD-323_HandSoldering, F.Cu at (177.2, 139.1)
- added D902: PESD5V0V1BA, Diode_SMD:D_SOD-323_HandSoldering, F.Cu at (172.1, 128.9)
- added D903: PESD5V0V1BA, Diode_SMD:D_SOD-323_HandSoldering, F.Cu at (168.9, 128.9)
- added D904: PESD5V0V1BA, Diode_SMD:D_SOD-323_HandSoldering, F.Cu at (165.7, 128.9)
- added D905: PESD5V0V1BA, Diode_SMD:D_SOD-323_HandSoldering, F.Cu at (162.6, 128.9)
- J1: footprint Video:6PinDIN240Degree -> CPCModular:6PinDIN240Degree
- JP1: value RC2014Bus -> CPCM_VideoRAM_EdgeBottom; footprint Connector_PinHeader_2.54mm:PinHeader_1x40_P2.54mm_Vertical -> CPCModular:Edge36_2.54PS; moved to B.Cu
- JP2: value RC2014ExtendedBus -> CPCM_VideoRAM_EdgeTop; footprint Connector_PinHeader_2.54mm:PinHeader_1x25_P2.54mm_Vertical -> CPCModular:Edge36_2.54PS
- moved X901 84.1 mm to (241.3, 108.0), turned to 270 degrees
- moved J1 79.2 mm to (165.1, 144.8), turned to 90 degrees
- moved R139 78.2 mm to (248.3, 144.1), turned to 90 degrees
- moved R138 76.1 mm to (244.5, 144.1), turned to 90 degrees
- moved R134 69.9 mm to (161.3, 116.2)
- moved R136 69.9 mm to (158.1, 123.8)
- moved Q102 67.3 mm to (162.6, 112.4), turned to 0 degrees
- moved R135 60.3 mm to (164.5, 116.2), turned to 270 degrees
- moved R137 54.0 mm to (167.6, 116.2), turned to 270 degrees
- moved IC118 53.0 mm to (214.0, 106.7), turned to 0 degrees
- moved JP2 41.8 mm to (158.8, 167.5)
- moved IC918 41.3 mm to (194.9, 106.7), turned to 0 degrees
- moved R133 40.0 mm to (178.4, 108.6), turned to 0 degrees
- moved R132 31.7 mm to (178.4, 118.1), turned to 0 degrees
- moved C104-2 30.1 mm to (233.0, 152.6), turned to 270 degrees
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Connections:
- net A10 renamed Net-(JP1-Pad6)
- net A11 renamed Net-(JP1-Pad5)
- net A12 renamed Net-(JP1-Pad4)
- net A2 renamed Net-(JP1-Pad14)
- net A3 renamed Net-(JP1-Pad13)
- net A4 renamed Net-(JP1-Pad12)
- net A5 renamed Net-(JP1-Pad11)
- net A6 renamed Net-(JP1-Pad10)
- net A7 renamed Net-(JP1-Pad9)
- net A8 renamed Net-(JP1-Pad8)
- net A9 renamed Net-(JP1-Pad7)
- IC118 pad 1: /1MHz -> /RAM_GA/~CPU_ADDR
- IC118 pad 12: /~ROMEN -> /RAM_GA/~ROMEN
- IC118 pad 13: /~RAMRD -> /RAM_GA/~RAMRD
- IC118 pad 15: /VSYNC -> /RAM_GA/VSYNC
- IC118 pad 24: RAMD0 -> RD0
- IC118 pad 25: RAMD1 -> RD1
- IC118 pad 26: RAMD2 -> RD2
- IC118 pad 27: RAMD3 -> RD3
- IC118 pad 28: RAMD4 -> RD4
- IC118 pad 29: RAMD5 -> RD5
- IC118 pad 30: RAMD6 -> RD6
- IC118 pad 31: RAMD7 -> RD7
- IC118 pad 6: /RAM_GA/GateArrays/~CAS_ADDR -> Net-(IC118-Pad6)
- IC918 pad 1: RAMD5 -> RD5
- IC918 pad 13: /VSYNC -> /RAM_GA/VSYNC
- IC918 pad 14: /1MHz -> /RAM_GA/~CPU_ADDR
- IC918 pad 2: RAMD6 -> RD6
- IC918 pad 27: /~ROMEN -> /RAM_GA/~ROMEN
- IC918 pad 29: /~RAMRD -> /RAM_GA/~RAMRD
- IC918 pad 3: RAMD7 -> RD7
- IC918 pad 31: /RAM_GA/GateArrays/~CAS_ADDR -> Net-(IC918-Pad31)
- IC918 pad 35: RAMD0 -> RD0
- IC918 pad 37: RAMD1 -> RD1
- IC918 pad 38: RAMD2 -> RD2
- IC918 pad 39: RAMD3 -> RD3
- IC918 pad 40: RAMD4 -> RD4
- JP1 pad 1: A15 -> GND
- JP1 pad 15: A1 -> /RAM_GA/~MREQ
- JP1 pad 16: A0 -> /RAM_GA/~RD
- JP1 pad 17: GND -> /RAM_GA/~ROMEN
- JP1 pad 18: +5V -> /RAM_GA/~RAMRD
- JP1 pad 19: /RAM_GA/~M1 -> Net-(JP1-Pad19)
- JP1 pad 2: A14 -> Net-(JP1-Pad2)
- JP1 pad 20: /RAM_GA/~RESET -> /RAM_GA/PHI
- JP1 pad 21: /RAM_GA/PHI -> /RAM_GA/MA0_CCLK
- JP1 pad 22: /RAM_GA/~INT -> /RAM_GA/~CAS
- JP1 pad 23: /RAM_GA/~MREQ -> /RAM_GA/~244EN
- JP1 pad 25: /RAM_GA/~RD -> /RAM_GA/~CPU_ADDR
- JP1 pad 26: /RAM_GA/~IORQ -> /RAM_GA/~RAS
- JP1 pad 27: Net-(JP1-Pad27) -> /RAM_GA/~MWE
- JP1 pad 3: A13 -> A14
- JP1 pad 32: Net-(JP1-Pad32) -> RD6
- JP1 pad 33: Net-(JP1-Pad33) -> RD4
- JP1 pad 34: Net-(JP1-Pad34) -> RD2
- JP1 pad 35: Net-(JP1-Pad35) -> RD0
- JP2 pad 1: GND -> Net-(JP2-Pad1)
- JP2 pad 11: RAMD0 -> Net-(JP2-Pad11)
- JP2 pad 12: RAMD1 -> Net-(JP2-Pad12)
- JP2 pad 13: RAMD2 -> Net-(JP2-Pad13)
- JP2 pad 14: RAMD3 -> Net-(JP2-Pad14)
- JP2 pad 15: RAMD4 -> +5V
- JP2 pad 16: RAMD5 -> /RAM_GA/~M1
- JP2 pad 17: RAMD6 -> /RAM_GA/~IORQ
- JP2 pad 18: RAMD7 -> Net-(JP2-Pad18)
- JP2 pad 19: Net-(JP2-Pad19) -> /RAM_GA/~INT
- JP2 pad 2: +5V -> Net-(JP2-Pad2)
- JP2 pad 20: Net-(JP2-Pad20) -> /RAM_GA/READY
- JP2 pad 21: Net-(JP2-Pad21) -> /RAM_GA/~RESET
- JP2 pad 22: /~RAMRD -> Net-(JP2-Pad22)
- JP2 pad 25: (no net) -> /RAM_GA/VSYNC
- JP2 pad 3: Net-(JP2-Pad3) -> A15
- JP2 pad 5: /1MHz -> Net-(JP2-Pad5)
- JP2 pad 9: /RAM_GA/READY -> Net-(JP2-Pad9)
Routing:
- net GND: track 85.0 -> 426.2 mm, vias 11 -> 1
- net +5V: track 25.2 -> 269.6 mm, vias 3 -> 0
- net RD5: track 0.00 -> 102.6 mm, vias 0 -> 3
- net RAMD5: track 100.1 -> 0.00 mm, vias 2 -> 0
- net RD6: track 0.00 -> 97.7 mm, vias 0 -> 4
- net RAMD6: track 97.0 -> 0.00 mm, vias 2 -> 0
- net RAMD7: track 97.0 -> 0.00 mm, vias 2 -> 0
- net RD7: track 0.00 -> 94.3 mm, vias 0 -> 3
- net RAMD4: track 92.1 -> 0.00 mm, vias 2 -> 0
- net RD0: track 0.00 -> 91.9 mm, vias 0 -> 3
- net RD1: track 0.00 -> 91.9 mm, vias 0 -> 2
- net RD3: track 0.00 -> 91.5 mm, vias 0 -> 2
- net RD4: track 0.00 -> 91.1 mm, vias 0 -> 3
- net RD2: track 0.00 -> 90.9 mm, vias 0 -> 3
- net /RAM_GA/MA0_CCLK: track 40.2 -> 130.8 mm, vias 0 -> 3
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- added copper zone on F.Cu, net GND
- removed copper zone on F.Cu, net +5V
Other:
- board size 99.1 x 52.9 mm -> 99.1 x 70.3 mm
- board text added: "An Amstrad CPC compatible computer."
- board text added: "Install (40007 or 40008) or 40010 but not both. R138, R139 only needed for 40007. Capacitors are 0.1uF unless noted otherwise. Diodes (D901..D905) are PESD5V0V1BA/SOD323, they are bidirectional so oritentation is irrelevant. The diodes are recommended for ESD protection but the board will work fine without them."
- board text added: "REV 2"
- board text added: "bread80.com github.com/Bread80 mstdn.social/@bread80"
- board text added: "© Mike Sutton, 2024 Bread80.com"
- board text removed: "A15 A14 A13 A12 A11 A10 A9 A8 A7 A6 A5 A4 A3 A2 A1 A0 Gnd 5v M1 Reset Clock INT Mreq Wr Ro IORQ D0 D1 D2 D3 D4 D5 D6 D7 Tx Rx USR1 USR2 USR3"
- board text removed: "An Amstrad CPC compatible using a (slightly modified) RC2014 backplane. This is NOT an RC2014 module."
- board text removed: "Install 40007 or 40008 in 'upper' socket, 40010 in 'lower' socket. R138, R139 only needed for 40007"
- board text removed: "Pin 1"
- board text removed: "REV 0.1"
- board text removed: "To RAM control board"
- board text removed: "bread80.com - mstdn.social/@bread80 gitgub.com/Bread80 - twitter.com/bread80com"
- board text removed: "© Mike Sutton, 2023 Bread80.com"
