File: Video/GateArrays.sch (KiCad schematic (older format))
At the start: 6 parts, among them IC118 AMG40007, IC918 AMG40010

Commit message: Long overdue update...
Connections:
- net ~CAS_ADDR: no longer names the net of IC118.6 (~CAS_ADDR)
- net ~CAS_ADDR: no longer IC918.31 (~CASAD)
- no-connect marks 0 -> 2
Changed lines of the file:
@@
 Text HLabel 1850 3200 0    50   Output ~ 0
 ~CPU_ADDR
-Text HLabel 1850 3300 0    50   Output ~ 0
-~CAS_ADDR
 Text HLabel 1850 3400 0    50   Output ~ 0
 MA0_CCLK
@@
 	1850 3200 1950 3200
 Wire Wire Line
-	1950 3300 1850 3300
-Wire Wire Line
 	1850 3400 1950 3400
 Wire Wire Line
@@
 Text HLabel 4900 3200 0    50   Output ~ 0
 ~CPU_ADDR
-Text HLabel 4900 3300 0    50   Output ~ 0
-~CAS_ADDR
 Text HLabel 4900 3400 0    50   Output ~ 0
 MA0_CCLK
@@
 	4900 3200 5000 3200
 Wire Wire Line
-	5000 3300 4900 3300
-Wire Wire Line
 	4900 3400 5000 3400
 Wire Wire Line
@@
 	1    0    0    -1
 $EndComp
+NoConn ~ 1950 3300
+NoConn ~ 5000 3300
 $EndSCHEMATC
