File: Video/RAM_GA.sch (KiCad schematic (older format))
At the start: 19 parts, among them J1 VIDEO OUT, Q102 2SC1815Y, Q103 2N2369, X201 16MHz CXO_DIP14

Commit message: Long overdue update...
Parts:
- added C139, C140, C141: 220p, Capacitor_THT:C_Disc_D3.0mm_W1.6mm_P2.50mm, symbol Device:C
- added C901: 1uF, Capacitor_THT:CP_Radial_D7.5mm_P2.50mm, symbol Device:CP
- added D901, D902, D903, D904, D905: PESD5V0V1BA, Diode_SMD:D_SOD-323_HandSoldering, symbol Device:D_TVS_ALT
- J1: footprint Video:6PinDIN240Degree -> CPCModular:6PinDIN240Degree
Connections:
- net +5V: now also C901.1
- net BLUE: now also C141.1, D903.2 (A2)
- net GND: now also C139.2, C140.2, C141.2, C901.2, D901.1 (A1), D902.1 (A1), D903.1 (A1), D904.1 (A1), D905.1 (A1)
- net GREEN: now also C140.1, D902.2 (A2)
- net LUM: now also D905.2 (A2)
- net RED: now also C139.1, D901.2 (A2)
- net ~SYNC: now also D904.2 (A2)
- no-connect marks 2 -> 1
Other:
- note added: "6-pin DIN, 240 degrees.\nE.g. TE 5786676-1"
- note added: "ESD Protection"
- moved on the sheet: J1, R136
